Commit message: Cleaned

File: stevie_description/urdf/macros.xacro (robot description, xacro)
@@ -29,17 +29,3 @@
 	  />
 	</xacro:macro>
-  <!-- creates a counterweight to move the center of mass of a link -->
-	<xacro:macro name="counterweight" params="parent m x y z">
-    <link name="${parent}_counterweight_link">
-			<inertial>
-				<mass value="${m}"/>
-				<inertia ixx="0.000001" ixy="0" ixz="0" iyy="0.000001" iyz="0" izz="0.000001"/>
-			</inertial>
-		</link>
-    <joint name="${parent}_counterweight_joint" type="fixed">
-			<origin xyz="${x} ${y} ${z}" rpy="0 0 0"/>
-			<parent link="${parent}"/>
-			<child link="${parent}_counterweight_link"/>
-		</joint>
-	</xacro:macro>
 </robot>
