Commit message: Controllers added and fonctionnal

File: stevie_description/urdf/arms/arms.transmission.xacro (robot description, xacro)
@@ -6,8 +6,8 @@
 			<type>transmission_interface/SimpleTransmission</type>
 			<joint name="upper_body_shoulder_${side}_joint">
-				<hardwareInterface>EffortJointInterface</hardwareInterface>
+				<hardwareInterface>hardware_interface/EffortJointInterface</hardwareInterface>
     		</joint>
 			<actuator name="shoulder_${side}_motor">
-				<hardwareInterface>EffortJointInterface</hardwareInterface>
+				<hardwareInterface>hardware_interface/EffortJointInterface</hardwareInterface>
 				<mechanicalReduction>1</mechanicalReduction>
 			</actuator>
@@ -18,9 +18,9 @@
 		<transmission name="arm_${side}_transmission">
 			<type>transmission_interface/SimpleTransmission</type>
-			<joint name="arm_${side}_joint">
-				<hardwareInterface>EffortJointInterface</hardwareInterface>
+			<joint name="shoulder_arm_${side}_joint">
+				<hardwareInterface>hardware_interface/EffortJointInterface</hardwareInterface>
     		</joint>
-			<actuator name="shoulder_arm_${side}_motor">
-				<hardwareInterface>EffortJointInterface</hardwareInterface>
+			<actuator name="arm_${side}_motor">
+				<hardwareInterface>hardware_interface/EffortJointInterface</hardwareInterface>
 				<mechanicalReduction>1</mechanicalReduction>
 			</actuator>

File: stevie_description/urdf/head/head.transmission.xacro (robot description, xacro)
@@ -4,13 +4,9 @@
 		<transmission name="neck_transmission">
 			<type>transmission_interface/SimpleTransmission</type>
-			<!-- FOR HYDRO -->  <!--
-			<joint name="wheel_${side}_joint"/>
-			-->
-			<!-- FOR INDIGO -->
 			<joint name="upper_body_neck_joint">
-				<hardwareInterface>EffortJointInterface</hardwareInterface>
+				<hardwareInterface>hardware_interface/EffortJointInterface</hardwareInterface>
     		</joint>
 			<actuator name="neck_motor">
-				<hardwareInterface>EffortJointInterface</hardwareInterface>
+				<hardwareInterface>hardware_interface/EffortJointInterface</hardwareInterface>
 				<mechanicalReduction>1</mechanicalReduction>
 			</actuator>
@@ -20,13 +16,9 @@
 		<transmission name="head_transmission">
 			<type>transmission_interface/SimpleTransmission</type>
-			<!-- FOR HYDRO -->  <!--
-			<joint name="wheel_${side}_joint"/>
-			-->
-			<!-- FOR INDIGO -->
 			<joint name="neck_head_joint">
-				<hardwareInterface>EffortJointInterface</hardwareInterface>
+				<hardwareInterface>hardware_interface/EffortJointInterface</hardwareInterface>
     		</joint>
 			<actuator name="head_motor">
-				<hardwareInterface>EffortJointInterface</hardwareInterface>
+				<hardwareInterface>hardware_interface/EffortJointInterface</hardwareInterface>
 				<mechanicalReduction>1</mechanicalReduction>
 			</actuator>

File: stevie_description/urdf/stevie.xacro (robot description, xacro)
@@ -1,28 +1,9 @@
 <?xml version="1.0"?>
 <robot name="stevie" xmlns:xacro="http://ros.org/wiki/xacro">
- <!--
-  <xacro:include filename="$(find robbie_description)/urdf/macros.xacro" />
-  <xacro:include filename="$(find robbie_description)/urdf/sensors/sensors.xacro" />
-  <xacro:include filename="$(find robbie_description)/urdf/robbie.gazebo"/>
--->
-	<!-- LOAD ROBOT COMPONENT FILES -->
-<!--
-  <xacro:include filename="$(find robbie_description)/urdf/shank/shank.xacro" />
-  <xacro:include filename="$(find robbie_description)/urdf/stabiliser/stabiliser.xacro" />
-  <xacro:include filename="$(find robbie_description)/urdf/thigh/thigh.xacro" />
-  <xacro:include filename="$(find robbie_description)/urdf/torso/torso.xacro" />
-  <xacro:include filename="$(find robbie_description)/urdf/lhm/lhm.xacro" />
-  <xacro:include filename="$(find robbie_description)/urdf/arm/arm.xacro" />
-	<xacro:shank_ass  name="shank"/>
-	<xacro:stabiliser parent="shank_link"/>
-	<xacro:thigh parent="shank_link" />
-	<xacro:torso parent="thigh_link" />
-	<xacro:lhm_ass/>
-	<xacro:arm_ass side="left" reflect="-1.0" arm_rotate="0.0" />
-	<xacro:arm_ass side="right" reflect="1.0" arm_rotate="1.0" />
--->
+  <xacro:include filename="$(find stevie_description)/urdf/macro.xacro" />
+  <xacro:include filename="$(find stevie_description)/urdf/stevie.gazebo"/>
+  <!-- LOAD ROBOT COMPONENT FILES -->
   <xacro:property name="lower_body_name" value="lower_body"/>
   <xacro:property name="upper_body_name" value="upper_body"/>
-  <xacro:include filename="$(find stevie_description)/urdf/macro.xacro" />
   <xacro:include filename="$(find stevie_description)/urdf/lower_body/lower_body.xacro" />
   <xacro:include filename="$(find stevie_description)/urdf/upper_body/upper_body.xacro" />

File: stevie_description/urdf/upper_body/hip.xacro (robot description, xacro)
@@ -50,5 +50,5 @@
 		</joint>
 		<!-- transmission -->
-		<xacro:hip_transmission parent="${parent}"/>
+		<xacro:hip_transmission/>
 	</xacro:macro>
 	<!--***********************************************************************-->

File: stevie_description/urdf/upper_body/upper_body.transmission.xacro (robot description, xacro)
@@ -2,12 +2,12 @@
 <robot xmlns:xacro="http://ros.org/wiki/xacro">
 	<!-- HIP -->
-	<xacro:macro name="hip_transmission" params="parent">
+	<xacro:macro name="hip_transmission">
 		<transmission name="hip_transmission">
 			<type>transmission_interface/SimpleTransmission</type>
-			<joint name="hip_${parent}_joint">
-				<hardwareInterface>EffortJointInterface</hardwareInterface>
+			<joint name="hip_lower_body_joint">
+				<hardwareInterface>hardware_interface/EffortJointInterface</hardwareInterface>
     		</joint>
 			<actuator name="hip_motor">
-				<hardwareInterface>EffortJointInterface</hardwareInterface>
+				<hardwareInterface>hardware_interface/EffortJointInterface</hardwareInterface>
 				<mechanicalReduction>1</mechanicalReduction>
 			</actuator>
@@ -15,12 +15,12 @@
 	</xacro:macro>
 	<!-- UPPER_BODY -->
-	<xacro:macro name="upper_body_transmission" params="name">
+	<xacro:macro name="upper_body_transmission">
 		<transmission name="upper_body_transmission">
 			<type>transmission_interface/SimpleTransmission</type>
-			<joint name="hip_${name}_joint">
-				<hardwareInterface>EffortJointInterface</hardwareInterface>
+			<joint name="upper_body_hip_joint">
+				<hardwareInterface>hardware_interface/EffortJointInterface</hardwareInterface>
     		</joint>
 			<actuator name="upper_body_motor">
-				<hardwareInterface>EffortJointInterface</hardwareInterface>
+				<hardwareInterface>hardware_interface/EffortJointInterface</hardwareInterface>
 				<mechanicalReduction>1</mechanicalReduction>
 			</actuator>

File: stevie_description/urdf/upper_body/upper_body.xacro (robot description, xacro)
@@ -51,5 +51,5 @@
 		</joint>
 		<!-- transmission -->
-		<xacro:upper_body_transmission name="${name}"/>
+		<xacro:upper_body_transmission/>
 	</xacro:macro>
 	<!--***********************************************************************-->

File: stevie_description/urdf/wheels/wheels.transmission.xacro (robot description, xacro)
@@ -5,8 +5,8 @@
 			<type>transmission_interface/SimpleTransmission</type>
 			<joint name="wheel_${side}_joint">
-				<hardwareInterface>EffortJointInterface</hardwareInterface>
+				<hardwareInterface>hardware_interface/EffortJointInterface</hardwareInterface>
     		</joint>
 			<actuator name="${side}_motor">
-				<hardwareInterface>EffortJointInterface</hardwareInterface>
+				<hardwareInterface>hardware_interface/EffortJointInterface</hardwareInterface>
 				<mechanicalReduction>1</mechanicalReduction>
 			</actuator>
