Commit message: Arms added

File: stevie_description/urdf/arms/arms.xacro (robot description, xacro)
@@ -4,4 +4,5 @@
 	<xacro:include filename="$(find stevie_description)/urdf/wheel/wheel.transmission.xacro" />
 -->
+	<xacro:include filename="$(find stevie_description)/urdf/arms/shoulders.xacro" />
 	<!-- DECLARE VARIABLES -->
 	<xacro:property name="arm_mass" value="1"/>
@@ -9,7 +10,13 @@
 	<xacro:property name="arm_width" value="0.1100"/>
 	<xacro:property name="arm_height" value="0.124658905"/>
+	<!--Adjust world's Y axis-->
+	<xacro:property name="arm_x_adjustment" value="0.065"/>
+	<!--Adjust world's -Z axis-->
+	<xacro:property name="right_arm_y_adjustment" value="-0.05"/>
+	<xacro:property name="left_arm_y_adjustment" value="0.55"/>
 	<xacro:property name="PI" value="3.14159"/>
 	<!--************************        ARMS          ************************-->
   <xacro:macro name="arm" params="parent side" >
+		<xacro:shoulder parent="${parent}" side="${side}"/>
 		<!-- arm link -->
 		<link name="arm_${side}_link">
@@ -48,12 +55,12 @@
 		<joint name="arm_${side}_joint" type="revolute">
 			<xacro:if value="${side == 'right'}">
-				<origin xyz="0 0 0" rpy="0 0 ${PI/2}"/>
+				<origin xyz="${arm_x_adjustment} ${right_arm_y_adjustment} 0" rpy="0 ${PI} ${PI}"/>
 			</xacro:if>
 			<xacro:if value="${side == 'left'}">
-				<origin xyz="0 0 0" rpy="0 0 ${-PI/2}"/>
+				<origin xyz="${arm_x_adjustment} ${left_arm_y_adjustment} 0" rpy="0 0 0"/>
 			</xacro:if>
 			<axis xyz="0 0 1"/>
 			<limit lower="-${PI/4}" upper="${PI/4}" effort="1000.0" velocity="0.5"/>
-			<parent link="${parent}"/>
+			<parent link="shoulder_${side}_link"/>
 			<child link="arm_${side}_link"/>
 		</joint>

File: stevie_description/urdf/arms/shoulders.xacro (robot description, xacro)
@@ -3,7 +3,4 @@
 <!--
 	<xacro:include filename="$(find stevie_description)/urdf/wheel/wheel.transmission.xacro" />
--->
-<!--
-	<xacro:include filename="$(find stevie_description)/urdf/arms/arms.xacro" />
 -->
 	<!-- DECLARE VARIABLES -->
@@ -42,10 +39,8 @@
 			<material>Gazebo/White</material>
 		</gazebo>
-		<!--*************   ARM     *************-->
-		<!--<xacro:arm parent="shoulder_${side}_link" side="${side}"/>-->
 		<!-- shoulder-arm joint -->
 		<joint name="shoulder_${side}_joint" type="revolute">
 			<xacro:if value="${side == 'right'}">
-				<origin xyz="${-upper_body_length/2 + shoulder_x_adjustment} ${upper_body_height + shoulder_y_adjustment} 0" rpy="${PI} ${PI} 0"/>
+				<origin xyz="${-upper_body_length/2 - shoulder_x_adjustment} ${upper_body_height + shoulder_y_adjustment} 0" rpy="${PI} ${PI} 0"/>
 			</xacro:if>
 			<xacro:if value="${side == 'left'}">

File: stevie_description/urdf/stevie.xacro (robot description, xacro)
@@ -26,7 +26,8 @@
   <xacro:include filename="$(find stevie_description)/urdf/lower_body/lower_body.xacro" />
   <xacro:include filename="$(find stevie_description)/urdf/upper_body/upper_body.xacro" />
-  <xacro:include filename="$(find stevie_description)/urdf/arms/shoulders.xacro" />
+  <xacro:include filename="$(find stevie_description)/urdf/arms/arms.xacro" />
   <xacro:lower_body  name="${lower_body_name}"/>
   <xacro:upper_body parent="${lower_body_name}_link" name="${upper_body_name}"/>
-  <xacro:shoulder parent="${upper_body_name}_link" side="left"/>
+  <xacro:arm parent="${upper_body_name}_link" side="left"/>
+  <xacro:arm parent="${upper_body_name}_link" side="right"/>
 </robot>

Commit message: Neck added + joint position correction + rotation axis correction

File: stevie_description/urdf/arms/arms.xacro (robot description, xacro)
@@ -12,7 +12,6 @@
 	<!--Adjust world's Y axis-->
 	<xacro:property name="arm_x_adjustment" value="0.065"/>
-	<!--Adjust world's -Z axis-->
-	<xacro:property name="right_arm_y_adjustment" value="-0.05"/>
-	<xacro:property name="left_arm_y_adjustment" value="0.55"/>
+	<!--Adjust world's Z axis-->
+	<xacro:property name="arm_link_y_adjustment" value="0.2"/>
 	<xacro:property name="PI" value="3.14159"/>
 	<!--************************        ARMS          ************************-->
@@ -55,11 +54,13 @@
 		<joint name="arm_${side}_joint" type="revolute">
 			<xacro:if value="${side == 'right'}">
-				<origin xyz="${arm_x_adjustment} ${right_arm_y_adjustment} 0" rpy="0 ${PI} ${PI}"/>
+				<origin xyz="${arm_x_adjustment} 0 0" rpy="0 ${PI} ${PI}"/>
+				<limit lower="0" upper="${PI/4}" effort="1000.0" velocity="0.5"/>
 			</xacro:if>
 			<xacro:if value="${side == 'left'}">
-				<origin xyz="${arm_x_adjustment} ${left_arm_y_adjustment} 0" rpy="0 0 0"/>
+				<!--<origin xyz="${arm_x_adjustment} ${-upper_body_height + left_arm_y_adjustment} 0" rpy="0 0 0"/>-->
+				<origin xyz="${arm_x_adjustment} 0 0" rpy="0 0 0"/>
+				<limit lower="${-PI/4}" upper="0" effort="1000.0" velocity="0.5"/>
 			</xacro:if>
 			<axis xyz="0 0 1"/>
-			<limit lower="-${PI/4}" upper="${PI/4}" effort="1000.0" velocity="0.5"/>
 			<parent link="shoulder_${side}_link"/>
 			<child link="arm_${side}_link"/>

File: stevie_description/urdf/arms/shoulders.xacro (robot description, xacro)
@@ -39,5 +39,5 @@
 			<material>Gazebo/White</material>
 		</gazebo>
-		<!-- shoulder-arm joint -->
+		<!-- upper_body-shoulder joint -->
 		<joint name="shoulder_${side}_joint" type="revolute">
 			<xacro:if value="${side == 'right'}">
@@ -47,5 +47,5 @@
 				<origin xyz="${upper_body_length/2 + shoulder_x_adjustment} ${upper_body_height + shoulder_y_adjustment} 0" rpy="${PI} 0 0"/>
 			</xacro:if>
-			<axis xyz="0 0 1"/>
+			<axis xyz="1 0 0"/>
 			<limit lower="-${PI/4}" upper="${PI/4}" effort="1000.0" velocity="0.5"/>
 			<parent link="${parent}"/>

File: stevie_description/urdf/stevie.xacro (robot description, xacro)
@@ -27,7 +27,9 @@
   <xacro:include filename="$(find stevie_description)/urdf/upper_body/upper_body.xacro" />
   <xacro:include filename="$(find stevie_description)/urdf/arms/arms.xacro" />
+  <xacro:include filename="$(find stevie_description)/urdf/head/neck.xacro" />
   <xacro:lower_body  name="${lower_body_name}"/>
   <xacro:upper_body parent="${lower_body_name}_link" name="${upper_body_name}"/>
   <xacro:arm parent="${upper_body_name}_link" side="left"/>
   <xacro:arm parent="${upper_body_name}_link" side="right"/>
+  <xacro:neck parent="${upper_body_name}_link"/>
 </robot>

File: stevie_description/urdf/upper_body/upper_body.xacro (robot description, xacro)
@@ -11,5 +11,6 @@
 	<xacro:property name="upper_body_height" value="0.565"/>
 	<!--Adjust the world's Z axis-->
-	<xacro:property name="upper_body_y_adjustment" value="0.049"/>
+	<xacro:property name="hip_upper_body_joint_y_adjustment" value="0.0733"/>
+	<xacro:property name="upper_body_link_y_adjustment" value="-0.024"/>
 	<xacro:property name="PI" value="3.14159"/>
 	<!--************************        UPPER BODY          ************************-->
@@ -18,5 +19,5 @@
 		<link name="${name}_link">
 			<collision>
-				<origin xyz="0 0 0" rpy="0 0 0"/>
+				<origin xyz="0 ${upper_body_link_y_adjustment} 0" rpy="0 0 0"/>
 				<geometry>
 					<mesh filename="package://stevie_description/meshes/collision/upper_body_collision.STL" scale="0.001 0.001 0.001"/>
@@ -24,5 +25,5 @@
 			</collision>
 			<visual>
-				<origin xyz="0 0 0" rpy="0 0 0"/>
+				<origin xyz="0 ${upper_body_link_y_adjustment} 0" rpy="0 0 0"/>
 					<geometry>
 				 		<mesh filename="package://stevie_description/meshes/visual/upper_body.STL" scale="0.001 0.001 0.001"/>
@@ -30,5 +31,5 @@
 			</visual>
 			<inertial>
-				<origin xyz="0 0 0" rpy="0 0 0"/>
+				<origin xyz="0 ${upper_body_link_y_adjustment} 0" rpy="0 0 0"/>
 				<mass value="${upper_body_mass}"/>
 				<inertia ixx="182592012288.0000" ixy="1131537.1250" ixz="-3420374.2500" iyy="137232130048.0000" iyz="-56384828.0000" izz="183043080192.0000"/>
@@ -42,6 +43,6 @@
 		<!-- hip-upper_body joint -->
 		<joint name="hip_${name}_joint" type="revolute">
-			<origin xyz="0 ${upper_body_y_adjustment} 0" rpy="0 0 0"/>
-			<axis xyz="0 0 1"/>
+			<origin xyz="0 ${hip_upper_body_joint_y_adjustment} 0" rpy="0 0 0"/>
+			<axis xyz="1 0 0"/>
 			<limit lower="-${PI/4}" upper="${PI/4}" effort="1000.0" velocity="0.5"/>
 			<parent link="hip_link"/>

File: stevie_description/urdf/wheels/wheels.xacro (robot description, xacro)
@@ -46,5 +46,5 @@
 			<parent link="${parent}"/>
 			<child link="wheel_${side}_link"/>
-			<axis xyz="0 1 0"/>
+			<axis xyz="1 0 0"/>
 		</joint>
 	</xacro:macro>

Commit message: Head added + origin relocated for some parts

File: stevie_description/urdf/arms/arms.xacro (robot description, xacro)
@@ -10,11 +10,8 @@
 	<xacro:property name="arm_width" value="0.1100"/>
 	<xacro:property name="arm_height" value="0.124658905"/>
-	<!--Adjust world's Y axis-->
-	<xacro:property name="arm_x_adjustment" value="0.065"/>
-	<!--Adjust world's Z axis-->
-	<xacro:property name="arm_link_y_adjustment" value="0.2"/>
 	<xacro:property name="PI" value="3.14159"/>
 	<!--************************        ARMS          ************************-->
   <xacro:macro name="arm" params="parent side" >
+		<!-- shoulder -->
 		<xacro:shoulder parent="${parent}" side="${side}"/>
 		<!-- arm link -->
@@ -27,5 +24,5 @@
 					</xacro:if>
 					<xacro:if value="${side == 'left'}">
-						<mesh filename="package://stevie_description/meshes/collision/left_arm_collision.STL" scale="0.001 0.001 0.001"/>
+						<mesh filename="package://stevie_description/meshes/collision/left_arm.STL" scale="0.001 0.001 0.001"/>
 					</xacro:if>
 				</geometry>
@@ -54,10 +51,9 @@
 		<joint name="arm_${side}_joint" type="revolute">
 			<xacro:if value="${side == 'right'}">
-				<origin xyz="${arm_x_adjustment} 0 0" rpy="0 ${PI} ${PI}"/>
+				<origin xyz="0 0 0" rpy="0 ${PI} ${PI}"/>
 				<limit lower="0" upper="${PI/4}" effort="1000.0" velocity="0.5"/>
 			</xacro:if>
 			<xacro:if value="${side == 'left'}">
-				<!--<origin xyz="${arm_x_adjustment} ${-upper_body_height + left_arm_y_adjustment} 0" rpy="0 0 0"/>-->
-				<origin xyz="${arm_x_adjustment} 0 0" rpy="0 0 0"/>
+				<origin xyz="0 0 0" rpy="0 0 0"/>
 				<limit lower="${-PI/4}" upper="0" effort="1000.0" velocity="0.5"/>
 			</xacro:if>

File: stevie_description/urdf/arms/shoulders.xacro (robot description, xacro)
@@ -10,7 +10,7 @@
 	<xacro:property name="shoulder_height" value="0.1150"/>
 	<!--Adjust world's Z axis-->
-	<xacro:property name="shoulder_y_adjustment" value="-0.1465"/>
+	<xacro:property name="shoulder_y_adjustment" value="-0.17"/>
 	<!--Adjust world's Y axis-->
-	<xacro:property name="shoulder_x_adjustment" value="-0.04"/>
+	<xacro:property name="shoulder_x_adjustment" value="0.035"/>
 	<xacro:property name="PI" value="3.14159"/>
 	<!--************************        SHOULDERS          ************************-->

File: stevie_description/urdf/head/neck.xacro (robot description, xacro)
@@ -10,5 +10,5 @@
 	<xacro:property name="neck_height" value="0.220"/>
 	<!--Adjust the world's Z axis-->
-	<xacro:property name="neck_y_adjustment" value="-0.065"/>
+	<xacro:property name="neck_y_adjustment" value="0.04"/>
 	<xacro:property name="PI" value="3.14159"/>
 	<!--************************        NECK          ************************-->

File: stevie_description/urdf/lower_body/lower_body.xacro (robot description, xacro)
@@ -7,5 +7,5 @@
 	<xacro:include filename="$(find stevie_description)/urdf/caster/caster.xacro" />
 	<!-- DECLARE VARIABLES -->
-	<xacro:property name="lower_body_mass" value="0.27"/>
+	<xacro:property name="lower_body_mass" value="27"/>
 	<xacro:property name="lower_body_length" value="0.485903015"/>
 	<xacro:property name="lower_body_width" value="0.516555237"/>
@@ -46,8 +46,8 @@
 			<child link="${name}_link"/>
 		</joint>
-		<!--**************        WHEELS          **************-->
+		<!-- wheels -->
 		<xacro:wheel parent="${name}_footprint" side="right"/>
 		<xacro:wheel parent="${name}_footprint" side="left"/>
-		<!--**************        CASTER          **************-->
+		<!-- caster wheel -->
 		<xacro:caster parent="${name}_footprint"/>
 	</xacro:macro>

File: stevie_description/urdf/stevie.xacro (robot description, xacro)
@@ -27,9 +27,9 @@
   <xacro:include filename="$(find stevie_description)/urdf/upper_body/upper_body.xacro" />
   <xacro:include filename="$(find stevie_description)/urdf/arms/arms.xacro" />
-  <xacro:include filename="$(find stevie_description)/urdf/head/neck.xacro" />
+  <xacro:include filename="$(find stevie_description)/urdf/head/head.xacro" />
   <xacro:lower_body  name="${lower_body_name}"/>
-  <xacro:upper_body parent="${lower_body_name}_link" name="${upper_body_name}"/>
+  <!--<xacro:upper_body parent="${lower_body_name}_link" name="${upper_body_name}"/>
   <xacro:arm parent="${upper_body_name}_link" side="left"/>
   <xacro:arm parent="${upper_body_name}_link" side="right"/>
-  <xacro:neck parent="${upper_body_name}_link"/>
+  <xacro:head parent="${upper_body_name}_link"/>-->
 </robot>

File: stevie_description/urdf/upper_body/hip.xacro (robot description, xacro)
@@ -12,5 +12,5 @@
 	<xacro:property name="hip_z_adjustment" value="-0.135"/>
 	<!--Adjust on the world's Z axis-->
-	<xacro:property name="hip_y_adjustment" value="-0.04"/>
+	<xacro:property name="hip_y_adjustment" value="0.025"/>
 	<xacro:property name="PI" value="3.14159"/>
 	<!--************************        HIP          ************************-->

File: stevie_description/urdf/upper_body/upper_body.xacro (robot description, xacro)
@@ -10,7 +10,4 @@
 	<xacro:property name="upper_body_width" value="0.283975830"/>
 	<xacro:property name="upper_body_height" value="0.565"/>
-	<!--Adjust the world's Z axis-->
-	<xacro:property name="hip_upper_body_joint_y_adjustment" value="0.0733"/>
-	<xacro:property name="upper_body_link_y_adjustment" value="-0.024"/>
 	<xacro:property name="PI" value="3.14159"/>
 	<!--************************        UPPER BODY          ************************-->
@@ -19,5 +16,5 @@
 		<link name="${name}_link">
 			<collision>
-				<origin xyz="0 ${upper_body_link_y_adjustment} 0" rpy="0 0 0"/>
+				<origin xyz="0 0 0" rpy="0 0 0"/>
 				<geometry>
 					<mesh filename="package://stevie_description/meshes/collision/upper_body_collision.STL" scale="0.001 0.001 0.001"/>
@@ -25,5 +22,5 @@
 			</collision>
 			<visual>
-				<origin xyz="0 ${upper_body_link_y_adjustment} 0" rpy="0 0 0"/>
+				<origin xyz="0 0 0" rpy="0 0 0"/>
 					<geometry>
 				 		<mesh filename="package://stevie_description/meshes/visual/upper_body.STL" scale="0.001 0.001 0.001"/>
@@ -31,5 +28,5 @@
 			</visual>
 			<inertial>
-				<origin xyz="0 ${upper_body_link_y_adjustment} 0" rpy="0 0 0"/>
+				<origin xyz="0 0 0" rpy="0 0 0"/>
 				<mass value="${upper_body_mass}"/>
 				<inertia ixx="182592012288.0000" ixy="1131537.1250" ixz="-3420374.2500" iyy="137232130048.0000" iyz="-56384828.0000" izz="183043080192.0000"/>
@@ -39,9 +36,9 @@
 			<material>Gazebo/White</material>
 		</gazebo>
-		<!--*************   HIP     *************-->
+		<!-- hip -->
 		<xacro:hip parent="${parent}"/>
 		<!-- hip-upper_body joint -->
 		<joint name="hip_${name}_joint" type="revolute">
-			<origin xyz="0 ${hip_upper_body_joint_y_adjustment} 0" rpy="0 0 0"/>
+			<origin xyz="0 0 0" rpy="0 0 0"/>
 			<axis xyz="1 0 0"/>
 			<limit lower="-${PI/4}" upper="${PI/4}" effort="1000.0" velocity="0.5"/>
