Commit message: Rotation applied to the different parts + corrected inertia and center of mass + macro to scale the inertia

File: stevie_description/urdf/arms/arms.xacro (robot description, xacro)
@@ -7,7 +7,10 @@
 	<!-- DECLARE VARIABLES -->
 	<xacro:property name="arm_mass" value="1"/>
+	<xacro:property name="arm_volume" value="0.002083"/>
 	<xacro:property name="arm_length" value="0.124658905"/>
 	<xacro:property name="arm_width" value="0.1100"/>
 	<xacro:property name="arm_height" value="0.124658905"/>
+	<xacro:property name="right_arm_center_of_mass" value="-0.001570 -0.001100 -0.074465"/>
+	<xacro:property name="left_arm_center_of_mass" value="-0.001570 0.001100 -0.074465"/>
 	<xacro:property name="PI" value="3.14159"/>
 	<!--************************        ARMS          ************************-->
@@ -20,10 +23,5 @@
 				<origin xyz="0 0 0" rpy="0 0 0"/>
 				<geometry>
-					<xacro:if value="${side == 'right'}">
-						<mesh filename="package://stevie_description/meshes/collision/right_arm_collision.STL" scale="0.001 0.001 0.001"/>
-					</xacro:if>
-					<xacro:if value="${side == 'left'}">
-						<mesh filename="package://stevie_description/meshes/collision/left_arm.STL" scale="0.001 0.001 0.001"/>
-					</xacro:if>
+					<mesh filename="package://stevie_description/meshes/collision/${side}_arm_collision.STL" scale="0.001 0.001 0.001"/>
 				</geometry>
 			</collision>
@@ -31,16 +29,17 @@
 				<origin xyz="0 0 0" rpy="0 0 0"/>
 				<geometry>
-					<xacro:if value="${side == 'right'}">
-						<mesh filename="package://stevie_description/meshes/visual/right_arm.STL" scale="0.001 0.001 0.001"/>
-					</xacro:if>
-					<xacro:if value="${side == 'left'}">
-						<mesh filename="package://stevie_description/meshes/visual/left_arm.STL" scale="0.001 0.001 0.001"/>
-					</xacro:if>
+					<mesh filename="package://stevie_description/meshes/visual/${side}_arm.STL" scale="0.001 0.001 0.001"/>
 				</geometry>
 			</visual>
 			<inertial>
-				<origin xyz="0 0 0" rpy="0 0 0"/>
+				<xacro:if value="${side == 'right'}">
+					<origin xyz="${right_arm_center_of_mass}" rpy="0 0 0"/>
+					<xacro:scale_inertia m="${arm_mass}" v="${arm_volume}" ixx="0.0000134861" ixy="-0.0000001570" ixz="-0.0000001100" iyy="0.0000140186" iyz="-0.0000000025" izz="0.0000028663"/>
+				</xacro:if>
+				<xacro:if value="${side == 'left'}">
+					<origin xyz="${left_arm_center_of_mass}" rpy="0 0 0"/>
+					<xacro:scale_inertia m="${arm_mass}" v="${arm_volume}" ixx="0.0000134861" ixy="0.0000000026" ixz="-0.0000001553" iyy="0.0000140187" iyz="0.0000000025" izz="0.0000028663"/>
+				</xacro:if>
 				<mass value="${arm_mass}"/>
-				<inertia ixx="14018668544.0000" ixy="2533231.2500" ixz="-2730643.5000" iyy="2866326016.0000" iyz="155359360.0000" izz="13486148608.0000"/>
 			</inertial>
 		</link>
@@ -51,12 +50,11 @@
 		<joint name="arm_${side}_joint" type="revolute">
 			<xacro:if value="${side == 'right'}">
-				<origin xyz="0 0 0" rpy="0 ${PI} ${PI}"/>
-				<limit lower="0" upper="${PI/4}" effort="1000.0" velocity="0.5"/>
+				<origin xyz="0 0 0" rpy="0 0 ${PI/2}"/>
 			</xacro:if>
 			<xacro:if value="${side == 'left'}">
-				<origin xyz="0 0 0" rpy="0 0 0"/>
-				<limit lower="${-PI/4}" upper="0" effort="1000.0" velocity="0.5"/>
+				<origin xyz="0 0 0" rpy="0 0 ${-PI/2}"/>
 			</xacro:if>
-			<axis xyz="0 0 1"/>
+			<limit lower="0" upper="${PI/4}" effort="1000.0" velocity="0.5"/>
+			<axis xyz="1 0 0"/>
 			<parent link="shoulder_${side}_link"/>
 			<child link="arm_${side}_link"/>

File: stevie_description/urdf/arms/shoulders.xacro (robot description, xacro)
@@ -6,11 +6,11 @@
 	<!-- DECLARE VARIABLES -->
 	<xacro:property name="shoulder_mass" value="1"/>
+	<xacro:property name="shoulder_volume" value="0.000678"/>
 	<xacro:property name="shoulder_length" value="0.2130"/>
 	<xacro:property name="shoulder_width" value="0.115000381"/>
 	<xacro:property name="shoulder_height" value="0.1150"/>
-	<!--Adjust world's Z axis-->
-	<xacro:property name="shoulder_y_adjustment" value="-0.17"/>
-	<!--Adjust world's Y axis-->
-	<xacro:property name="shoulder_x_adjustment" value="0.035"/>
+	<xacro:property name="shoulder_center_of_mass" value="-0.023361 0 0.002146"/>
+	<xacro:property name="shoulder_z_adjustment" value="-0.17"/>
+	<xacro:property name="shoulder_y_adjustment" value="0.035"/>
 	<xacro:property name="PI" value="3.14159"/>
 	<!--************************        SHOULDERS          ************************-->
@@ -31,7 +31,7 @@
 			</visual>
 			<inertial>
-				<origin xyz="0 0 0" rpy="0 0 0"/>
+				<origin xyz="${shoulder_center_of_mass}" rpy="0 0 0"/>
 				<mass value="${shoulder_mass}"/>
-				<inertia ixx="822072832.0000" ixy="-14428306.0000" ixz="7534.551758" iyy="1594399616.0000" iyz="-3097.950439" izz="1878856192.0000"/>
+				<xacro:scale_inertia m="${shoulder_mass}" v="${shoulder_volume}" ixx="0.0000008220" ixy="0.0000000000" ixz="0.0000000144" iyy="0.0000018788" iyz="0.0000000000" izz="0.0000015944"/>
 			</inertial>
 		</link>
@@ -42,10 +42,11 @@
 		<joint name="shoulder_${side}_joint" type="revolute">
 			<xacro:if value="${side == 'right'}">
-				<origin xyz="${-upper_body_length/2 - shoulder_x_adjustment} ${upper_body_height + shoulder_y_adjustment} 0" rpy="${PI} ${PI} 0"/>
+				<origin xyz="0 ${-upper_body_length/2 - shoulder_y_adjustment} ${upper_body_height + shoulder_z_adjustment}" rpy="0 0 ${-PI/2}"/>
+				<axis xyz="1 0 0"/>
 			</xacro:if>
 			<xacro:if value="${side == 'left'}">
-				<origin xyz="${upper_body_length/2 + shoulder_x_adjustment} ${upper_body_height + shoulder_y_adjustment} 0" rpy="${PI} 0 0"/>
+				<origin xyz="0 ${upper_body_length/2 + shoulder_y_adjustment} ${upper_body_height + shoulder_z_adjustment}" rpy="0 0 ${PI/2}"/>
+				<axis xyz="-1 0 0"/>
 			</xacro:if>
-			<axis xyz="1 0 0"/>
 			<limit lower="-${PI/4}" upper="${PI/4}" effort="1000.0" velocity="0.5"/>
 			<parent link="${parent}"/>

File: stevie_description/urdf/caster/caster.xacro (robot description, xacro)
@@ -47,5 +47,5 @@
 		<!-- footprint-caster joint -->
 		<joint name="caster_joint" type="fixed">
-			<origin xyz="${caster_x_adjustment} 0 ${caster_z_adjustment}" rpy="${PI/2} 0 0"/>
+			<origin xyz="${caster_x_adjustment} 0 ${caster_z_adjustment}" rpy="0 0 0"/>
 			<parent link="${parent}"/>
 			<child link="caster_link"/>

File: stevie_description/urdf/head/head.xacro (robot description, xacro)
@@ -11,4 +11,10 @@
 	<xacro:property name="head_height" value="0.300608185"/>
 	<xacro:property name="PI" value="3.14159"/>
+	<xacro:macro name="box_inertia" params="m x y z">
+    <inertia  ixx="${m*(y*y+z*z)/12}" ixy="0" ixz="0"
+              iyy="${m*(x*x+z*z)/12}" iyz="0"
+              izz="${m*(x*x+z*z)/12}"
+    />
+  </xacro:macro>
 	<!--************************        HEAD          ************************-->
   <xacro:macro name="head" params="parent" >
@@ -30,7 +36,7 @@
 			</visual>
 			<inertial>
-				<origin xyz="0 0 0" rpy="0 0 0"/>
+				<origin xyz="0 0 ${head_height / 2}" rpy="0 0 0"/>
 				<mass value="${head_mass}"/>
-				<inertia ixx="119192846336.0000" ixy="15985847296.0000" ixz="2580351.2500" iyy="99658653696.0000" iyz="15342592.0000" izz="107701559296.0000"/>
+				<xacro:box_inertia m="${head_mass}" x="${head_width}" y="${head_height}" z="${head_length}"/>
 			</inertial>
 		</link>
@@ -40,6 +46,6 @@
 		<!-- neck-head joint -->
 		<joint name="neck_head_joint" type="revolute">
-			<origin xyz="0 0 0" rpy="0 ${-PI/2} 0"/>
-			<axis xyz="0 0 1"/>
+			<origin xyz="0 0 0" rpy="0 0 0"/>
+			<axis xyz="0 1 0"/>
 			<limit lower="-${PI/4}" upper="${PI/4}" effort="1000.0" velocity="0.5"/>
 			<parent link="neck_link"/>

File: stevie_description/urdf/head/neck.xacro (robot description, xacro)
@@ -6,9 +6,11 @@
 	<!-- DECLARE VARIABLES -->
 	<xacro:property name="neck_mass" value="0.5"/>
+	<xacro:property name="neck_volume" value="0.00073"/>
 	<xacro:property name="neck_length" value="0.110"/>
 	<xacro:property name="neck_width" value="0.110"/>
 	<xacro:property name="neck_height" value="0.220"/>
+	<xacro:property name="neck_center_of_mass" value="0 0 -0.095837"/>
 	<!--Adjust the world's Z axis-->
-	<xacro:property name="neck_y_adjustment" value="0.04"/>
+	<xacro:property name="neck_z_adjustment" value="0.04"/>
 	<xacro:property name="PI" value="3.14159"/>
 	<!--************************        NECK          ************************-->
@@ -29,7 +31,7 @@
 			</visual>
 			<inertial>
-				<origin xyz="0 0 0" rpy="0 0 0"/>
+				<origin xyz="${neck_center_of_mass}" rpy="0 0 0"/>
 				<mass value="${neck_mass}"/>
-				<inertia ixx="1929662464.0000" ixy="0.0" ixz="-1.590871" iyy="619161024.0000" iyz="0.0" izz="1930710144.0000"/>
+				<xacro:scale_inertia m="${neck_mass}" v="${neck_volume}" ixx="0.000019307" ixy="0.000000" ixz="0.000000" iyy="0.0000019296" iyz="0.000000" izz="0.0000006191"/>
 			</inertial>
 		</link>
@@ -39,6 +41,6 @@
 		<!-- upper_body-neck joint -->
 		<joint name="upper_body_neck_joint" type="revolute">
-			<origin xyz="0 ${upper_body_height + neck_y_adjustment} 0" rpy="0 0 0"/>
-			<axis xyz="0 1 0"/>
+			<origin xyz="0 0 ${upper_body_height + neck_z_adjustment}" rpy="0 0 0"/>
+			<axis xyz="0 0 1"/>
 			<limit lower="-${PI/4}" upper="${PI/4}" effort="1000.0" velocity="0.5"/>
 			<parent link="${parent}"/>

File: stevie_description/urdf/lower_body/lower_body.xacro (robot description, xacro)
@@ -6,11 +6,19 @@
 	<xacro:include filename="$(find stevie_description)/urdf/wheels/wheels.xacro" />
 	<xacro:include filename="$(find stevie_description)/urdf/caster/caster.xacro" />
+	<xacro:include filename="$(find stevie_description)/urdf/macro.xacro" />
 	<!-- DECLARE VARIABLES -->
 	<xacro:property name="lower_body_mass" value="27"/>
-	<xacro:property name="lower_body_length" value="0.485903015"/>
-	<xacro:property name="lower_body_width" value="0.516555237"/>
+	<xacro:property name="lower_body_volume" value="0.016607"/>
+	<xacro:property name="lower_body_length" value="0.485903"/>
+	<xacro:property name="lower_body_width" value="0.516555"/>
 	<xacro:property name="lower_body_height" value="0.475"/>
-	<xacro:property name="lower_body_z_adjustment" value="-0.075"/>
+	<xacro:property name="lower_body_center_of_mass" value="-0.112043 0.000001 0.051805"/>
 	<xacro:property name="PI" value="3.14159"/>
+	<xacro:macro name="box_inertia" params="m x y z">
+    <inertia  ixx="${m*(y*y+z*z)/12}" ixy="0" ixz="0"
+              iyy="${m*(x*x+z*z)/12}" iyz="0"
+              izz="${m*(x*x+z*z)/12}"
+    />
+  </xacro:macro>
 	<!--************************        LOWER BODY          ************************-->
   <xacro:macro name="lower_body" params="name" >
@@ -32,7 +40,7 @@
 			</visual>
 			<inertial>
-				<origin xyz="0 0 0" rpy="0 0 0"/>
+				<origin xyz="${lower_body_center_of_mass}" rpy="0 0 0"/>
 				<mass value="${lower_body_mass}"/>
-				<inertia ixx="405031911424.0000" ixy="-6338355.0000" ixz="1364738.3750" iyy="423088029696.0000" iyz="3831503104.0000" izz="255725256704.0000"/>
+				<xacro:scale_inertia m="${lower_body_mass}" v="${lower_body_volume}" ixx="0.0002557254" ixy="0.0000000013" ixz="0.0000038315" iyy="0.0004050320" iyz="-0.00000000634" izz="0.0004230882"/>
 			</inertial>
 		</link>
@@ -40,10 +48,41 @@
 			<material>Gazebo/White</material>
 		</gazebo>
+<!--
+	<link name="${name}_link">
+		<collision>
+			<origin xyz="0 0 0.2" rpy="0 0 0"/>
+			<geometry>
+				<box size="${lower_body_length} ${lower_body_width - 0.2} ${lower_body_height}"/>
+			</geometry>
+		</collision>
+		<visual>
+			<origin xyz="0 0 0.2" rpy="0 0 0"/>
+				<geometry>
+					<box size="${lower_body_length} ${lower_body_width - 0.2} ${lower_body_height}"/>
+				</geometry>
+		</visual>
+		<inertial>
+			<origin xyz="0 0 0.2" rpy="0 0 0"/>
+			<mass value="${lower_body_mass}"/>
+			<box_inertia m="${lower_body_mass}" x="${lower_body_length}" y="${lower_body_width - 0.2}" z="${lower_body_height}"/>
+		</inertial>
+	</link>
+	<gazebo reference="${name}_link">
+		<material>Gazebo/White</material>
+	</gazebo>
+-->
 		<!-- footprint-lower_body joint -->
 		<joint name="${name}_footprint_joint" type="fixed">
-			<origin xyz="0 0 ${lower_body_z_adjustment}" rpy="${PI/2} 0 ${PI/2}"/>
+			<origin xyz="0 0 ${wheel_radius / 2}" rpy="0 0 0"/>
 			<parent link="${name}_footprint"/>
 			<child link="${name}_link"/>
 		</joint>
+<!--
+	<joint name="${name}_footprint_joint" type="fixed">
+		<origin xyz="0 0 0" rpy="0 0 0"/>
+		<parent link="${name}_footprint"/>
+		<child link="${name}_link"/>
+	</joint>
+-->
 		<!-- wheels -->
 		<xacro:wheel parent="${name}_footprint" side="right"/>

File: stevie_description/urdf/stevie.xacro (robot description, xacro)
@@ -29,7 +29,7 @@
   <xacro:include filename="$(find stevie_description)/urdf/head/head.xacro" />
   <xacro:lower_body  name="${lower_body_name}"/>
-  <!--<xacro:upper_body parent="${lower_body_name}_link" name="${upper_body_name}"/>
+  <xacro:upper_body parent="${lower_body_name}_link" name="${upper_body_name}"/>
   <xacro:arm parent="${upper_body_name}_link" side="left"/>
   <xacro:arm parent="${upper_body_name}_link" side="right"/>
-  <xacro:head parent="${upper_body_name}_link"/>-->
+  <xacro:head parent="${upper_body_name}_link"/>
 </robot>

File: stevie_description/urdf/upper_body/hip.xacro (robot description, xacro)
@@ -4,13 +4,14 @@
 	<xacro:include filename="$(find stevie_description)/urdf/hip/hip.transmission.xacro" />
 -->
+	<xacro:include filename="$(find stevie_description)/urdf/macro.xacro" />
 	<!-- DECLARE VARIABLES -->
 	<xacro:property name="hip_mass" value="0.1"/>
+	<xacro:property name="hip_volume" value="0.001004"/>
 	<xacro:property name="hip_length" value="0.320"/>
 	<xacro:property name="hip_width" value="0.095"/>
 	<xacro:property name="hip_height" value="0.3"/>
-	<!--Adjust on the world's X axis-->
-	<xacro:property name="hip_z_adjustment" value="-0.135"/>
-	<!--Adjust on the world's Z axis-->
-	<xacro:property name="hip_y_adjustment" value="0.025"/>
+	<xacro:property name="hip_center_of_mass" value="0 0 -0.056289"/>
+	<xacro:property name="hip_x_adjustment" value="-0.135"/>
+	<xacro:property name="hip_z_adjustment" value="0.43"/>
 	<xacro:property name="PI" value="3.14159"/>
 	<!--************************        HIP          ************************-->
@@ -31,7 +32,7 @@
 			</visual>
 			<inertial>
-				<origin xyz="0 0 0" rpy="0 0 0"/>
+				<origin xyz="${hip_center_of_mass}" rpy="0 0 0"/>
 				<mass value="${hip_mass}"/>
-				<inertia ixx="6483752960.0000" ixy="2350.257568" ixz="-355.673645" iyy="14856898560.0000" iyz="-228.070938" izz="9096541184.0000"/>
+				<xacro:scale_inertia m="${hip_mass}" v="${hip_volume}" ixx="0.0000090965" ixy="0" ixz="0" iyy="0.0000064837" iyz="0" izz="0.0000148569"/>
 			</inertial>
 		</link>
@@ -41,7 +42,7 @@
 		<!-- lower_body-hip joint -->
 		<joint name="hip_${parent}_joint" type="revolute">
-			<origin xyz="0 ${lower_body_height + hip_y_adjustment} ${hip_z_adjustment}" rpy="0 0 0"/>
-			<axis xyz="0 1 0"/>
-			<limit lower="-${PI/2}" upper="${PI/2}" effort="1000.0" velocity="0.5"/>
+			<origin xyz="${hip_x_adjustment} 0 ${hip_z_adjustment}" rpy="0 0 0"/>
+			<axis xyz="0 0 1"/>
+			<limit lower="-${PI/4}" upper="${PI/4}" effort="1000.0" velocity="0.5"/>
 			<parent link="${parent}"/>
 			<child link="hip_link"/>

File: stevie_description/urdf/upper_body/upper_body.xacro (robot description, xacro)
@@ -7,7 +7,9 @@
 	<!-- DECLARE VARIABLES -->
 	<xacro:property name="upper_body_mass" value="8"/>
+	<xacro:property name="upper_body_volume" value="0.010712"/>
 	<xacro:property name="upper_body_length" value="0.347374786"/>
 	<xacro:property name="upper_body_width" value="0.283975830"/>
 	<xacro:property name="upper_body_height" value="0.565"/>
+	<xacro:property name="upper_body_center_of_mass" value="0.000090 0 0.390377"/>
 	<xacro:property name="PI" value="3.14159"/>
 	<!--************************        UPPER BODY          ************************-->
@@ -28,7 +30,7 @@
 			</visual>
 			<inertial>
-				<origin xyz="0 0 0" rpy="0 0 0"/>
+				<origin xyz="${upper_body_center_of_mass}" rpy="0 0 0"/>
 				<mass value="${upper_body_mass}"/>
-				<inertia ixx="182592012288.0000" ixy="1131537.1250" ixz="-3420374.2500" iyy="137232130048.0000" iyz="-56384828.0000" izz="183043080192.0000"/>
+				<xacro:scale_inertia m="${upper_body_mass}" v="${upper_body_volume}" ixx="0.0001825920" ixy="0" ixz="0" iyy="0.0001372321" iyz="0" izz="0.0001830431"/>
 			</inertial>
 		</link>
@@ -41,6 +43,6 @@
 		<joint name="hip_${name}_joint" type="revolute">
 			<origin xyz="0 0 0" rpy="0 0 0"/>
-			<axis xyz="1 0 0"/>
-			<limit lower="-${PI/4}" upper="${PI/4}" effort="1000.0" velocity="0.5"/>
+			<axis xyz="0 1 0"/>
+			<limit lower="-${PI/6}" upper="${PI/6}" effort="1000.0" velocity="0.5"/>
 			<parent link="hip_link"/>
 			<child link="${name}_link"/>

File: stevie_description/urdf/wheels/wheels.xacro (robot description, xacro)
@@ -6,9 +6,16 @@
 	<!-- DECLARE VARIABLES -->
 	<xacro:property name="wheel_mass" value="1"/>
-	<xacro:property name="wheel_radius" value="0.10125"/>
-	<xacro:property name="wheel_thickness" value="0.04800"/>
+	<xacro:property name="wheel_radius" value="0.101238"/>
+	<xacro:property name="wheel_thickness" value="0.045983"/>
 	<xacro:property name="wheel_box_length" value="0.110775482"/>
-	<xacro:property name="chassis_length" value="0.3032"/>
+	<xacro:property name="chassis_length" value="0.303032"/>
+	<xacro:property name="chassis_width" value="0.5"/>
 	<xacro:property name="PI" value="3.14159"/>
+	<xacro:macro name="cylinder_inertia" params="m r h">
+	  <inertia  ixx="${m*(3*r*r+h*h)/12}" ixy = "0" ixz = "0"
+	    iyy="${m*(3*r*r+h*h)/12}" iyz = "0"
+	    izz="${m*r*r/2}"
+	  />
+	</xacro:macro>
 	<!--************************        WHEELS          ************************-->
   <xacro:macro name="wheel" params="parent side" >
@@ -28,10 +35,15 @@
 			</visual>
 			<inertial>
-				<origin xyz="0 0 0" rpy="0 0 0"/>
+				<origin xyz="0 0 0" rpy="0 ${PI/2} 0"/>
 				<mass value="${wheel_mass}"/>
-				<inertia ixx="7694243840.0000" ixy="21.275770" ixz="47.828678" iyy="4313382912.0000" iyz="65.004593" izz="4313351168.0000"/>
+				<xacro:cylinder_inertia m="${wheel_mass}" r="${wheel_radius}" h="${wheel_thickness}"/>
 			</inertial>
 		</link>
 		<gazebo reference="wheel_${side}_link">
+			<mu1>1.0</mu1>
+			<mu2>1.0</mu2>
+			<kp value="10000000.0"/>
+      <kd value="1.0"/>
+      <fdir1 value="1 0 0"/>
 			<material>Gazebo/Black</material>
 		</gazebo>
@@ -40,11 +52,14 @@
 			<xacro:if value="${side == 'right'}">
 				<origin xyz="0 ${- wheel_thickness - chassis_length/2} 0" rpy="0 0 ${PI/2}"/>
+				<axis xyz="1 0 0"/>
 			</xacro:if>
 			<xacro:if value="${side == 'left'}">
 				<origin xyz="0 ${wheel_thickness + chassis_length/2} 0" rpy="0 0 ${-PI/2}"/>
+				<axis xyz="-1 0 0"/>
 			</xacro:if>
 			<parent link="${parent}"/>
 			<child link="wheel_${side}_link"/>
-			<axis xyz="1 0 0"/>
+      <limit effort="100" velocity="100"/>
+      <joint_properties damping="0.0" friciton="0.5"/>
 		</joint>
 	</xacro:macro>
