Commit message: Correction of limits and correction of link relations

File: stevie_description/urdf/arms/arms.xacro (robot description, xacro)
@@ -51,12 +51,14 @@
 			<xacro:if value="${side == 'right'}">
 				<origin xyz="0 0 0" rpy="0 0 ${PI/2}"/>
+				<limit lower="${-PI/4}" upper="0" effort="1000.0" velocity="0.5"/>
 			</xacro:if>
 			<xacro:if value="${side == 'left'}">
 				<origin xyz="0 0 0" rpy="0 0 ${-PI/2}"/>
+				<limit lower="0" upper="${PI/4}" effort="1000.0" velocity="0.5"/>
 			</xacro:if>
-			<limit lower="0" upper="${PI/4}" effort="1000.0" velocity="0.5"/>
 			<axis xyz="1 0 0"/>
 			<parent link="shoulder_${side}_link"/>
 			<child link="arm_${side}_link"/>
+      <joint_properties damping="10" friciton="0.5"/>
 		</joint>
 	</xacro:macro>

File: stevie_description/urdf/arms/shoulders.xacro (robot description, xacro)
@@ -52,4 +52,5 @@
 			<parent link="${parent}"/>
 			<child link="shoulder_${side}_link"/>
+      <joint_properties damping="10" friciton="0.5"/>
 		</joint>
 	</xacro:macro>

File: stevie_description/urdf/head/head.xacro (robot description, xacro)
@@ -51,4 +51,5 @@
 			<parent link="neck_link"/>
 			<child link="head_link"/>
+      <joint_properties damping="10" friciton="0.5"/>
 		</joint>
 	</xacro:macro>

File: stevie_description/urdf/head/neck.xacro (robot description, xacro)
@@ -46,4 +46,6 @@
 			<parent link="${parent}"/>
 			<child link="neck_link"/>
+      <limit effort="100" velocity="100"/>
+      <joint_properties damping="10" friciton="0.5"/>
 		</joint>
 	</xacro:macro>

File: stevie_description/urdf/lower_body/lower_body.xacro (robot description, xacro)
@@ -6,5 +6,4 @@
 	<xacro:include filename="$(find stevie_description)/urdf/wheels/wheels.xacro" />
 	<xacro:include filename="$(find stevie_description)/urdf/caster/caster.xacro" />
-	<xacro:include filename="$(find stevie_description)/urdf/macro.xacro" />
 	<!-- DECLARE VARIABLES -->
 	<xacro:property name="lower_body_mass" value="27"/>
@@ -15,10 +14,4 @@
 	<xacro:property name="lower_body_center_of_mass" value="-0.112043 0.000001 0.051805"/>
 	<xacro:property name="PI" value="3.14159"/>
-	<xacro:macro name="box_inertia" params="m x y z">
-    <inertia  ixx="${m*(y*y+z*z)/12}" ixy="0" ixz="0"
-              iyy="${m*(x*x+z*z)/12}" iyz="0"
-              izz="${m*(x*x+z*z)/12}"
-    />
-  </xacro:macro>
 	<!--************************        LOWER BODY          ************************-->
   <xacro:macro name="lower_body" params="name" >
@@ -48,46 +41,15 @@
 			<material>Gazebo/White</material>
 		</gazebo>
-<!--
-	<link name="${name}_link">
-		<collision>
-			<origin xyz="0 0 0.2" rpy="0 0 0"/>
-			<geometry>
-				<box size="${lower_body_length} ${lower_body_width - 0.2} ${lower_body_height}"/>
-			</geometry>
-		</collision>
-		<visual>
-			<origin xyz="0 0 0.2" rpy="0 0 0"/>
-				<geometry>
-					<box size="${lower_body_length} ${lower_body_width - 0.2} ${lower_body_height}"/>
-				</geometry>
-		</visual>
-		<inertial>
-			<origin xyz="0 0 0.2" rpy="0 0 0"/>
-			<mass value="${lower_body_mass}"/>
-			<box_inertia m="${lower_body_mass}" x="${lower_body_length}" y="${lower_body_width - 0.2}" z="${lower_body_height}"/>
-		</inertial>
-	</link>
-	<gazebo reference="${name}_link">
-		<material>Gazebo/White</material>
-	</gazebo>
--->
 		<!-- footprint-lower_body joint -->
 		<joint name="${name}_footprint_joint" type="fixed">
-			<origin xyz="0 0 ${wheel_radius / 2}" rpy="0 0 0"/>
+			<origin xyz="0 0 0" rpy="0 0 0"/>
 			<parent link="${name}_footprint"/>
 			<child link="${name}_link"/>
 		</joint>
-<!--
-	<joint name="${name}_footprint_joint" type="fixed">
-		<origin xyz="0 0 0" rpy="0 0 0"/>
-		<parent link="${name}_footprint"/>
-		<child link="${name}_link"/>
-	</joint>
--->
 		<!-- wheels -->
-		<xacro:wheel parent="${name}_footprint" side="right"/>
-		<xacro:wheel parent="${name}_footprint" side="left"/>
+		<xacro:wheel parent="${name}_link" side="right"/>
+		<xacro:wheel parent="${name}_link" side="left"/>
 		<!-- caster wheel -->
-		<xacro:caster parent="${name}_footprint"/>
+		<xacro:caster parent="${name}_link"/>
 	</xacro:macro>
 	<!--***********************************************************************-->

File: stevie_description/urdf/stevie.xacro (robot description, xacro)
@@ -24,4 +24,5 @@
   <xacro:property name="lower_body_name" value="lower_body"/>
   <xacro:property name="upper_body_name" value="upper_body"/>
+  <xacro:include filename="$(find stevie_description)/urdf/macro.xacro" />
   <xacro:include filename="$(find stevie_description)/urdf/lower_body/lower_body.xacro" />
   <xacro:include filename="$(find stevie_description)/urdf/upper_body/upper_body.xacro" />
@@ -30,6 +31,6 @@
   <xacro:lower_body  name="${lower_body_name}"/>
   <xacro:upper_body parent="${lower_body_name}_link" name="${upper_body_name}"/>
-  <xacro:arm parent="${upper_body_name}_link" side="left"/>
+  <!--<xacro:arm parent="${upper_body_name}_link" side="left"/>
   <xacro:arm parent="${upper_body_name}_link" side="right"/>
-  <xacro:head parent="${upper_body_name}_link"/>
+  <xacro:head parent="${upper_body_name}_link"/><-->
 </robot>

File: stevie_description/urdf/upper_body/hip.xacro (robot description, xacro)
@@ -4,5 +4,4 @@
 	<xacro:include filename="$(find stevie_description)/urdf/hip/hip.transmission.xacro" />
 -->
-	<xacro:include filename="$(find stevie_description)/urdf/macro.xacro" />
 	<!-- DECLARE VARIABLES -->
 	<xacro:property name="hip_mass" value="0.1"/>
@@ -47,4 +46,5 @@
 			<parent link="${parent}"/>
 			<child link="hip_link"/>
+      <joint_properties damping="10" friciton="0.5"/>
 		</joint>
 	</xacro:macro>

File: stevie_description/urdf/upper_body/upper_body.xacro (robot description, xacro)
@@ -47,4 +47,5 @@
 			<parent link="hip_link"/>
 			<child link="${name}_link"/>
+      <joint_properties damping="10" friciton="0.5"/>
 		</joint>
 	</xacro:macro>

File: stevie_description/urdf/wheels/wheels.xacro (robot description, xacro)
@@ -48,5 +48,5 @@
 			<material>Gazebo/Black</material>
 		</gazebo>
-		<!-- footprint-wheel joint -->
+		<!-- lower_body-wheel joint -->
 		<joint name="wheel_${side}_joint" type="continuous">
 			<xacro:if value="${side == 'right'}">

Commit message: Transmission added

File: stevie_description/urdf/arms/arms.xacro (robot description, xacro)
@@ -1,4 +1,4 @@
 <?xml version="1.0"?>
-<robot  xmlns:xacro="http://www.ros.org/wiki/xacro">
+<robot  xmlns:xacro="http://ros.org/wiki/xacro">
 <!--
 	<xacro:include filename="$(find stevie_description)/urdf/wheel/wheel.transmission.xacro" />
@@ -48,5 +48,5 @@
 		</gazebo>
 		<!-- shoulder-arm joint -->
-		<joint name="arm_${side}_joint" type="revolute">
+		<joint name="shoulder_arm_${side}_joint" type="revolute">
 			<xacro:if value="${side == 'right'}">
 				<origin xyz="0 0 0" rpy="0 0 ${PI/2}"/>
@@ -62,4 +62,6 @@
       <joint_properties damping="10" friciton="0.5"/>
 		</joint>
+		<!-- transmission -->
+		<xacro:arm_transmission side="${side}"/>
 	</xacro:macro>
 	<!--***********************************************************************-->

File: stevie_description/urdf/arms/shoulders.xacro (robot description, xacro)
@@ -1,4 +1,4 @@
 <?xml version="1.0"?>
-<robot  xmlns:xacro="http://www.ros.org/wiki/xacro">
+<robot  xmlns:xacro="http://ros.org/wiki/xacro">
 <!--
 	<xacro:include filename="$(find stevie_description)/urdf/wheel/wheel.transmission.xacro" />
@@ -40,5 +40,5 @@
 		</gazebo>
 		<!-- upper_body-shoulder joint -->
-		<joint name="shoulder_${side}_joint" type="revolute">
+		<joint name="upper_body_shoulder_${side}_joint" type="revolute">
 			<xacro:if value="${side == 'right'}">
 				<origin xyz="0 ${-upper_body_length/2 - shoulder_y_adjustment} ${upper_body_height + shoulder_z_adjustment}" rpy="0 0 ${-PI/2}"/>
@@ -54,4 +54,6 @@
       <joint_properties damping="10" friciton="0.5"/>
 		</joint>
+		<!-- transmission -->
+		<xacro:shoulder_transmission side="${side}"/>
 	</xacro:macro>
 	<!--***********************************************************************-->

File: stevie_description/urdf/caster/caster.xacro (robot description, xacro)
@@ -1,4 +1,4 @@
 <?xml version="1.0"?>
-<robot  xmlns:xacro="http://www.ros.org/wiki/xacro">
+<robot  xmlns:xacro="http://ros.org/wiki/xacro">
 <!--
 	<xacro:include filename="$(find stevie_description)/urdf/wheel/wheel.transmission.xacro" />

File: stevie_description/urdf/head/head.xacro (robot description, xacro)
@@ -1,7 +1,5 @@
 <?xml version="1.0"?>
-<robot  xmlns:xacro="http://www.ros.org/wiki/xacro">
-<!--
-	<xacro:include filename="$(find stevie_description)/urdf/hip/hip.transmission.xacro" />
--->
+<robot  xmlns:xacro="http://ros.org/wiki/xacro">
+	<xacro:include filename="$(find stevie_description)/urdf/head/head.transmission.xacro" />
 	<xacro:include filename="$(find stevie_description)/urdf/head/neck.xacro" />
 	<!-- DECLARE VARIABLES -->
@@ -53,4 +51,6 @@
       <joint_properties damping="10" friciton="0.5"/>
 		</joint>
+		<!-- transmission -->
+		<xacro:head_transmission/>
 	</xacro:macro>
 	<!--***********************************************************************-->

File: stevie_description/urdf/head/neck.xacro (robot description, xacro)
@@ -1,4 +1,4 @@
 <?xml version="1.0"?>
-<robot  xmlns:xacro="http://www.ros.org/wiki/xacro">
+<robot  xmlns:xacro="http://ros.org/wiki/xacro">
 <!--
 	<xacro:include filename="$(find stevie_description)/urdf/hip/hip.transmission.xacro" />
@@ -49,4 +49,6 @@
       <joint_properties damping="10" friciton="0.5"/>
 		</joint>
+		<!-- transmission -->
+		<xacro:neck_transmission/>
 	</xacro:macro>
 	<!--***********************************************************************-->

File: stevie_description/urdf/lower_body/lower_body.xacro (robot description, xacro)
@@ -1,4 +1,4 @@
 <?xml version="1.0"?>
-<robot  xmlns:xacro="http://www.ros.org/wiki/xacro">
+<robot  xmlns:xacro="http://ros.org/wiki/xacro">
 <!--
 	<xacro:include filename="$(find stevie_description)/urdf/lower_body/lower_body.transmission.xacro" />

File: stevie_description/urdf/macro.xacro (robot description, xacro)
@@ -1,4 +1,4 @@
 <?xml version="1.0"?>
-<robot  xmlns:xacro="http://www.ros.org/wiki/xacro">
+<robot  xmlns:xacro="http://ros.org/wiki/xacro">
   <xacro:macro name="scale_inertia" params="m v ixx ixy ixz iyy iyz izz" >
 		<inertia 	ixx="${ixx * m / v}" 	ixy="${ixy * m / v}" 	ixz="${ixz * m / v}"

File: stevie_description/urdf/stevie.xacro (robot description, xacro)
@@ -1,4 +1,4 @@
 <?xml version="1.0"?>
-<robot name="stevie" xmlns:xacro="http://www.ros.org/wiki/xacro">
+<robot name="stevie" xmlns:xacro="http://ros.org/wiki/xacro">
  <!--
   <xacro:include filename="$(find robbie_description)/urdf/macros.xacro" />

File: stevie_description/urdf/upper_body/hip.xacro (robot description, xacro)
@@ -1,7 +1,5 @@
 <?xml version="1.0"?>
-<robot  xmlns:xacro="http://www.ros.org/wiki/xacro">
-<!--
-	<xacro:include filename="$(find stevie_description)/urdf/hip/hip.transmission.xacro" />
--->
+<robot  xmlns:xacro="http://ros.org/wiki/xacro">
+	<xacro:include filename="$(find stevie_description)/urdf/upper_body/upper_body.transmission.xacro" />
 	<!-- DECLARE VARIABLES -->
 	<xacro:property name="hip_mass" value="0.1"/>
@@ -48,4 +46,6 @@
       <joint_properties damping="10" friciton="0.5"/>
 		</joint>
+		<!-- transmission -->
+		<xacro:hip_transmission parent="${parent}"/>
 	</xacro:macro>
 	<!--***********************************************************************-->

File: stevie_description/urdf/upper_body/upper_body.xacro (robot description, xacro)
@@ -1,7 +1,5 @@
 <?xml version="1.0"?>
-<robot  xmlns:xacro="http://www.ros.org/wiki/xacro">
-<!--
-	<xacro:include filename="$(find stevie_description)/urdf/hip/hip.transmission.xacro" />
--->
+<robot  xmlns:xacro="http://ros.org/wiki/xacro">
+	<xacro:include filename="$(find stevie_description)/urdf/upper_body/upper_body.transmission.xacro" />
 	<xacro:include filename="$(find stevie_description)/urdf/upper_body/hip.xacro" />
 	<!-- DECLARE VARIABLES -->
@@ -49,4 +47,6 @@
       <joint_properties damping="10" friciton="0.5"/>
 		</joint>
+		<!-- transmission -->
+		<xacro:upper_body_transmission name="${name}"/>
 	</xacro:macro>
 	<!--***********************************************************************-->

File: stevie_description/urdf/wheels/wheels.transmission.xacro (robot description, xacro)
@@ -2,14 +2,10 @@
 <robot xmlns:xacro="http://ros.org/wiki/xacro">
 	<xacro:macro name="wheel_transmission" params="side">
-		<transmission name="${side}_transmission">
+		<transmission name="wheel_${side}_transmission">
 			<type>transmission_interface/SimpleTransmission</type>
-			<!-- FOR HYDRO -->  <!--
-			<joint name="wheel_${side}_joint"/>
-			-->
-			<!-- FOR INDIGO -->
 			<joint name="wheel_${side}_joint">
 				<hardwareInterface>EffortJointInterface</hardwareInterface>
     		</joint>
-			<actuator name="${side}_Motor">
+			<actuator name="${side}_motor">
 				<hardwareInterface>EffortJointInterface</hardwareInterface>
 				<mechanicalReduction>1</mechanicalReduction>

File: stevie_description/urdf/wheels/wheels.xacro (robot description, xacro)
@@ -1,7 +1,5 @@
 <?xml version="1.0"?>
-<robot  xmlns:xacro="http://www.ros.org/wiki/xacro">
-<!--
-	<xacro:include filename="$(find stevie_description)/urdf/wheel/wheel.transmission.xacro" />
--->
+<robot  xmlns:xacro="http://ros.org/wiki/xacro">
+	<xacro:include filename="$(find stevie_description)/urdf/wheels/wheels.transmission.xacro" />
 	<!-- DECLARE VARIABLES -->
 	<xacro:property name="wheel_mass" value="1"/>
@@ -63,4 +61,6 @@
       <joint_properties damping="0.0" friciton="0.5"/>
 		</joint>
+		<!-- transmission -->
+		<xacro:wheel_transmission side="${side}"/>
 	</xacro:macro>
 	<!--***********************************************************************-->

Commit message: Controllers added

File: stevie_description/urdf/arms/arms.xacro (robot description, xacro)
@@ -47,5 +47,5 @@
 			<mu1>1.0</mu1>
 			<mu2>1.0</mu2>
-			<maxVel value="0"/>
+			<maxVel>0</maxVel>
 			<material>Gazebo/White</material>
 		</gazebo>

File: stevie_description/urdf/arms/shoulders.xacro (robot description, xacro)
@@ -37,5 +37,5 @@
 			<mu1>1.0</mu1>
 			<mu2>1.0</mu2>
-			<maxVel value="0"/>
+			<maxVel>0</maxVel>
 			<material>Gazebo/White</material>
 		</gazebo>

File: stevie_description/urdf/caster/caster.xacro (robot description, xacro)
@@ -31,5 +31,5 @@
 				<origin xyz="0 0 0" rpy="0 0 0"/>
 				<geometry>
-					<mesh filename="package://stevie_description/meshes/collision/caster_collision.STL" scale="0.001 0.001 0.001"/>
+					<mesh filename="package://stevie_description/meshes/visual/caster.STL" scale="0.001 0.001 0.001"/>
 				</geometry>
 			</visual>
@@ -43,5 +43,5 @@
 			<mu1>0.0</mu1>
 			<mu2>0.0</mu2>
-			<maxVel value="0"/>
+			<maxVel>0</maxVel>
 			<material>Gazebo/Black</material>
 		</gazebo>

File: stevie_description/urdf/head/head.xacro (robot description, xacro)
@@ -42,5 +42,5 @@
 			<mu1>1.0</mu1>
 			<mu2>1.0</mu2>
-			<maxVel value="0"/>
+			<maxVel>0</maxVel>
 			<material>Gazebo/White</material>
 		</gazebo>

File: stevie_description/urdf/head/neck.xacro (robot description, xacro)
@@ -39,5 +39,5 @@
 			<mu1>1.0</mu1>
 			<mu2>1.0</mu2>
-			<maxVel value="0"/>
+			<maxVel>0</maxVel>
 			<material>Gazebo/White</material>
 		</gazebo>

File: stevie_description/urdf/lower_body/lower_body.xacro (robot description, xacro)
@@ -41,5 +41,5 @@
 			<mu1>1.0</mu1>
 			<mu2>1.0</mu2>
-			<maxVel value="0"/>
+			<maxVel>0</maxVel>
 			<material>Gazebo/White</material>
 		</gazebo>

File: stevie_description/urdf/upper_body/hip.xacro (robot description, xacro)
@@ -37,9 +37,9 @@
 			<mu1>1.0</mu1>
 			<mu2>1.0</mu2>
-			<maxVel value="0"/>
+			<maxVel>0</maxVel>
 			<material>Gazebo/White</material>
 		</gazebo>
 		<!-- lower_body-hip joint -->
-		<joint name="hip_${parent}_joint" type="revolute">
+		<joint name="hip_lower_body_joint" type="revolute">
 			<origin xyz="${hip_x_adjustment} 0 ${hip_z_adjustment}" rpy="0 0 0"/>
 			<axis xyz="0 0 1"/>

File: stevie_description/urdf/upper_body/upper_body.xacro (robot description, xacro)
@@ -36,11 +36,11 @@
 			<mu1>1.0</mu1>
 			<mu2>1.0</mu2>
-			<maxVel value="0"/>
+			<maxVel>0</maxVel>
 			<material>Gazebo/White</material>
 		</gazebo>
 		<!-- hip -->
 		<xacro:hip parent="${parent}"/>
-		<!-- hip-upper_body joint -->
-		<joint name="hip_${name}_joint" type="revolute">
+		<!-- upper_body-hip joint -->
+		<joint name="upper_body_hip_joint" type="revolute">
 			<origin xyz="0 0 0" rpy="0 0 0"/>
 			<axis xyz="0 1 0"/>

File: stevie_description/urdf/wheels/wheels.xacro (robot description, xacro)
@@ -29,5 +29,5 @@
 				<origin xyz="0 0 0" rpy="0 0 0"/>
 				<geometry>
-					<mesh filename="package://stevie_description/meshes/collision/wheel_collision.STL" scale="0.001 0.001 0.001"/>
+					<mesh filename="package://stevie_description/meshes/visual/wheel.STL" scale="0.001 0.001 0.001"/>
 				</geometry>
 			</visual>
@@ -44,5 +44,5 @@
       <kd value="1.0"/>
       <fdir1 value="1 0 0"/>
-			<maxVel value="0"/>
+			<maxVel>0</maxVel>
 			<material>Gazebo/Black</material>
 		</gazebo>

Commit message: Stable robot

File: stevie_description/urdf/arms/arms.xacro (robot description, xacro)
@@ -63,5 +63,5 @@
 			<parent link="shoulder_${side}_link"/>
 			<child link="arm_${side}_link"/>
-      <joint_properties damping="10" friciton="0.5"/>
+      <dynamics damping="10" friction="0.5"/>
 		</joint>
 		<!-- transmission -->

File: stevie_description/urdf/arms/shoulders.xacro (robot description, xacro)
@@ -53,5 +53,5 @@
 			<parent link="${parent}"/>
 			<child link="shoulder_${side}_link"/>
-      <joint_properties damping="10" friciton="0.5"/>
+      <dynamics damping="10" friction="0.5"/>
 		</joint>
 		<!-- transmission -->

File: stevie_description/urdf/head/head.xacro (robot description, xacro)
@@ -46,5 +46,5 @@
 			<parent link="neck_link"/>
 			<child link="head_link"/>
-      <joint_properties damping="10" friciton="0.5"/>
+      <dynamics damping="10" friction="0.5"/>
 		</joint>
 		<!-- transmission -->

File: stevie_description/urdf/head/neck.xacro (robot description, xacro)
@@ -50,5 +50,5 @@
 			<child link="neck_link"/>
       <limit effort="100" velocity="100"/>
-      <joint_properties damping="10" friciton="0.5"/>
+      <dynamics damping="10" friction="0.5"/>
 		</joint>
 		<!-- transmission -->

File: stevie_description/urdf/upper_body/hip.xacro (robot description, xacro)
@@ -44,8 +44,8 @@
 			<origin xyz="${hip_x_adjustment} 0 ${hip_z_adjustment}" rpy="0 0 0"/>
 			<axis xyz="0 0 1"/>
-			<limit lower="-${PI/4}" upper="${PI/4}" effort="1000.0" velocity="0.5"/>
+			<limit lower="${-PI/4}" upper="${PI/4}" effort="1000.0" velocity="0.5"/>
 			<parent link="${parent}"/>
 			<child link="hip_link"/>
-      <joint_properties damping="10" friciton="0.5"/>
+      <dynamics damping="10" friction="0.5"/>
 		</joint>
 		<!-- transmission -->

File: stevie_description/urdf/upper_body/upper_body.xacro (robot description, xacro)
@@ -45,8 +45,8 @@
 			<origin xyz="0 0 0" rpy="0 0 0"/>
 			<axis xyz="0 1 0"/>
-			<limit lower="-${PI/6}" upper="${PI/6}" effort="1000.0" velocity="0.5"/>
+			<limit lower="${-PI/4}" upper="${PI/4}" effort="1000.0" velocity="0.5"/>
 			<parent link="hip_link"/>
 			<child link="${name}_link"/>
-      <joint_properties damping="10" friciton="0.5"/>
+      <dynamics damping="10" friction="1.5"/>
 		</joint>
 		<!-- transmission -->

File: stevie_description/urdf/wheels/wheels.xacro (robot description, xacro)
@@ -54,5 +54,5 @@
 			<child link="wheel_${side}_link"/>
       <limit effort="100" velocity="100"/>
-      <joint_properties damping="0.0" friciton="0.5"/>
+      <dynamics damping="0.0" friction="0.5"/>
 		</joint>
 		<!-- transmission -->
