Commit message: STL extension changed to stl. Wheel caps, screens and earcovers added

File: stevie_description/urdf/arms/arms.xacro (robot description, xacro)
@@ -23,5 +23,5 @@
 				<origin xyz="0 0 0" rpy="0 0 0"/>
 				<geometry>
-					<mesh filename="package://stevie_description/meshes/collision/${side}_arm_collision.STL" scale="0.001 0.001 0.001"/>
+					<mesh filename="package://stevie_description/meshes/collision/${side}_arm_collision.stl" scale="0.001 0.001 0.001"/>
 				</geometry>
 			</collision>
@@ -29,5 +29,5 @@
 				<origin xyz="0 0 0" rpy="0 0 0"/>
 				<geometry>
-					<mesh filename="package://stevie_description/meshes/visual/${side}_arm.STL" scale="0.001 0.001 0.001"/>
+					<mesh filename="package://stevie_description/meshes/visual/${side}_arm.stl" scale="0.001 0.001 0.001"/>
 				</geometry>
 			</visual>

File: stevie_description/urdf/arms/shoulders.xacro (robot description, xacro)
@@ -19,5 +19,5 @@
 				<origin xyz="0 0 0" rpy="0 0 0"/>
 				<geometry>
-					<mesh filename="package://stevie_description/meshes/collision/shoulder_collision.STL" scale="0.001 0.001 0.001"/>
+					<mesh filename="package://stevie_description/meshes/collision/shoulder_collision.stl" scale="0.001 0.001 0.001"/>
 				</geometry>
 			</collision>
@@ -25,5 +25,5 @@
 				<origin xyz="0 0 0" rpy="0 0 0"/>
 				<geometry>
-					<mesh filename="package://stevie_description/meshes/visual/shoulder.STL" scale="0.001 0.001 0.001"/>
+					<mesh filename="package://stevie_description/meshes/visual/shoulder.stl" scale="0.001 0.001 0.001"/>
 				</geometry>
 			</visual>

File: stevie_description/urdf/caster/caster.xacro (robot description, xacro)
@@ -31,5 +31,5 @@
 				<origin xyz="0 0 0" rpy="0 0 0"/>
 				<geometry>
-					<mesh filename="package://stevie_description/meshes/visual/caster.STL" scale="0.001 0.001 0.001"/>
+					<mesh filename="package://stevie_description/meshes/visual/caster.stl" scale="0.001 0.001 0.001"/>
 				</geometry>
 			</visual>

File: stevie_description/urdf/head/head.xacro (robot description, xacro)
@@ -18,5 +18,5 @@
 				<origin xyz="0 0 0" rpy="0 0 0"/>
 				<geometry>
-					<mesh filename="package://stevie_description/meshes/collision/head_collision.STL" scale="0.001 0.001 0.001"/>
+					<mesh filename="package://stevie_description/meshes/collision/head_collision.stl" scale="0.001 0.001 0.001"/>
 				</geometry>
 			</collision>
@@ -24,5 +24,5 @@
 				<origin xyz="0 0 0" rpy="0 0 0"/>
 					<geometry>
-				 		<mesh filename="package://stevie_description/meshes/visual/head.STL" scale="0.001 0.001 0.001"/>
+				 		<mesh filename="package://stevie_description/meshes/visual/head.stl" scale="0.001 0.001 0.001"/>
 					</geometry>
 			</visual>
@@ -50,4 +50,75 @@
 		<!-- transmission -->
 		<xacro:head_transmission/>
+		<!--************************        SCREENS          ************************-->
+		<!-- upper screen link -->
+		<link name="upper_screen_link">
+			<visual>
+				<origin xyz="0 0 0" rpy="0 0 0"/>
+				<geometry>
+					<mesh filename="package://stevie_description/meshes/visual/upper_screen.stl" scale="0.001001 0.001001 0.001001"/>
+				</geometry>
+			</visual>
+			<inertial>
+				<origin xyz="0 0 0" rpy="0 ${PI/2} 0"/>
+				<mass value="0.00001"/>
+				<inertia ixx="1.0" ixy="0" ixz="0" iyy="1.0" iyz="0" izz="1.0"/>
+			</inertial>
+		</link>
+		<gazebo reference="upper_screen_link">
+			<material>Gazebo/Black</material>
+		</gazebo>
+		<!-- upper_screen joint -->
+		<joint name="upper_screen_joint" type="fixed">
+			<origin xyz="0 0 0" rpy="0 0 0"/>
+			<parent link="head_link"/>
+			<child link="upper_screen_link"/>
+		</joint>
+		<!-- lower screen link -->
+		<link name="lower_screen_link">
+			<visual>
+				<origin xyz="0 0 0" rpy="0 0 0"/>
+				<geometry>
+					<mesh filename="package://stevie_description/meshes/visual/lower_screen.stl" scale="0.001001 0.001001 0.001001"/>
+				</geometry>
+			</visual>
+			<inertial>
+				<origin xyz="0 0 0" rpy="0 ${PI/2} 0"/>
+				<mass value="0.00001"/>
+				<inertia ixx="1.0" ixy="0" ixz="0" iyy="1.0" iyz="0" izz="1.0"/>
+			</inertial>
+		</link>
+		<gazebo reference="lower_screen_link">
+			<material>Gazebo/Black</material>
+		</gazebo>
+		<!-- lower_screen joint -->
+		<joint name="lower_screen_joint" type="fixed">
+			<origin xyz="0 0 0" rpy="0 0 0"/>
+			<parent link="head_link"/>
+			<child link="lower_screen_link"/>
+		</joint>
+		<!--************************        EARCOVERS          ************************-->
+		<!-- earcovers link -->
+		<link name="earcovers_link">
+			<visual>
+				<origin xyz="0 0 0" rpy="0 0 0"/>
+				<geometry>
+					<mesh filename="package://stevie_description/meshes/visual/earcovers.stl" scale="0.001 0.001 0.001"/>
+				</geometry>
+			</visual>
+			<inertial>
+				<origin xyz="0 0 0" rpy="0 ${PI/2} 0"/>
+				<mass value="0.00001"/>
+				<inertia ixx="1.0" ixy="0" ixz="0" iyy="1.0" iyz="0" izz="1.0"/>
+			</inertial>
+		</link>
+		<gazebo reference="earcovers_link">
+			<material>Gazebo/Yellow</material>
+		</gazebo>
+		<!-- upper_screen joint -->
+		<joint name="earcovers_joint" type="fixed">
+			<origin xyz="0 0 0" rpy="0 0 0"/>
+			<parent link="head_link"/>
+			<child link="earcovers_link"/>
+		</joint>
 	</xacro:macro>
 	<!--***********************************************************************-->

File: stevie_description/urdf/head/neck.xacro (robot description, xacro)
@@ -21,5 +21,5 @@
 				<origin xyz="0 0 0" rpy="0 0 0"/>
 				<geometry>
-					<mesh filename="package://stevie_description/meshes/collision/neck_collision.STL" scale="0.001 0.001 0.001"/>
+					<mesh filename="package://stevie_description/meshes/collision/neck_collision.stl" scale="0.001 0.001 0.001"/>
 				</geometry>
 			</collision>
@@ -27,5 +27,5 @@
 				<origin xyz="0 0 0" rpy="0 0 0"/>
 					<geometry>
-				 		<mesh filename="package://stevie_description/meshes/visual/neck.STL" scale="0.001 0.001 0.001"/>
+				 		<mesh filename="package://stevie_description/meshes/visual/neck.stl" scale="0.001 0.001 0.001"/>
 					</geometry>
 			</visual>

File: stevie_description/urdf/lower_body/lower_body.xacro (robot description, xacro)
@@ -23,5 +23,5 @@
 				<origin xyz="0 0 0" rpy="0 0 0"/>
 				<geometry>
-					<mesh filename="package://stevie_description/meshes/collision/lower_body_collision.STL" scale="0.001 0.001 0.001"/>
+					<mesh filename="package://stevie_description/meshes/collision/lower_body_collision.stl" scale="0.001 0.001 0.001"/>
 				</geometry>
 			</collision>
@@ -29,5 +29,5 @@
 				<origin xyz="0 0 0" rpy="0 0 0"/>
 					<geometry>
-				 		<mesh filename="package://stevie_description/meshes/visual/lower_body.STL" scale="0.001 0.001 0.001"/>
+				 		<mesh filename="package://stevie_description/meshes/visual/lower_body.stl" scale="0.001 0.001 0.001"/>
 					</geometry>
 			</visual>

File: stevie_description/urdf/upper_body/hip.xacro (robot description, xacro)
@@ -19,5 +19,5 @@
 				<origin xyz="0 0 0" rpy="0 0 0"/>
 				<geometry>
-					<mesh filename="package://stevie_description/meshes/collision/hip_upper_collision.STL" scale="0.001 0.001 0.001"/>
+					<mesh filename="package://stevie_description/meshes/collision/hip_upper_collision.stl" scale="0.001 0.001 0.001"/>
 				</geometry>
 			</collision>
@@ -25,5 +25,5 @@
 				<origin xyz="0 0 0" rpy="0 0 0"/>
 					<geometry>
-				 		<mesh filename="package://stevie_description/meshes/visual/hip_upper.STL" scale="0.001 0.001 0.001"/>
+				 		<mesh filename="package://stevie_description/meshes/visual/hip_upper.stl" scale="0.001 0.001 0.001"/>
 					</geometry>
 			</visual>

File: stevie_description/urdf/upper_body/upper_body.xacro (robot description, xacro)
@@ -18,12 +18,12 @@
 				<origin xyz="0 0 0" rpy="0 0 0"/>
 				<geometry>
-					<mesh filename="package://stevie_description/meshes/collision/upper_body_collision.STL" scale="0.001 0.001 0.001"/>
+					<mesh filename="package://stevie_description/meshes/collision/upper_body_collision.stl" scale="0.001 0.001 0.001"/>
 				</geometry>
 			</collision>
 			<visual>
 				<origin xyz="0 0 0" rpy="0 0 0"/>
-					<geometry>
-				 		<mesh filename="package://stevie_description/meshes/visual/upper_body.STL" scale="0.001 0.001 0.001"/>
-					</geometry>
+				<geometry>
+			 		<mesh filename="package://stevie_description/meshes/visual/upper_body.stl" scale="0.001 0.001 0.001"/>
+				</geometry>
 			</visual>
 			<inertial>

File: stevie_description/urdf/wheels/wheels.xacro (robot description, xacro)
@@ -23,5 +23,5 @@
 				<origin xyz="0 0 0" rpy="0 0 0"/>
 				<geometry>
-					<mesh filename="package://stevie_description/meshes/visual/wheel.STL" scale="0.001 0.001 0.001"/>
+					<mesh filename="package://stevie_description/meshes/visual/wheel.stl" scale="0.001 0.001 0.001"/>
 				</geometry>
 			</visual>
@@ -58,4 +58,29 @@
 		<!-- transmission -->
 		<xacro:wheel_transmission side="${side}"/>
+		<!--************************        WHEEL CAPS          ************************-->
+		<!-- wheel cap link -->
+		<link name="wheel_cap_${side}_link">
+			<visual>
+				<origin xyz="0 0 0" rpy="0 0 0"/>
+				<geometry>
+					<!-- slightly larger scale so the yellow cap can cover the one already on the wheel mesh -->
+					<mesh filename="package://stevie_description/meshes/visual/wheel_cap.stl" scale="0.001001 0.001001 0.001001"/>
+				</geometry>
+			</visual>
+			<inertial>
+				<origin xyz="0 0 0" rpy="0 ${PI/2} 0"/>
+				<mass value="0.00001"/>
+				<inertia ixx="1.0" ixy="0" ixz="0" iyy="1.0" iyz="0" izz="1.0"/>
+			</inertial>
+		</link>
+		<gazebo reference="wheel_cap_${side}_link">
+			<material>Gazebo/Yellow</material>
+		</gazebo>
+		<!-- wheel_cap joint -->
+		<joint name="wheel_cap_${side}_joint" type="fixed">
+			<origin xyz="0 0 0" rpy="0 0 0"/>
+			<parent link="wheel_${side}_link"/>
+			<child link="wheel_cap_${side}_link"/>
+		</joint>
 	</xacro:macro>
 	<!--***********************************************************************-->

Commit message: Arm sphere added + inertia corrected

File: stevie_description/urdf/arms/arms.xacro (robot description, xacro)
@@ -10,5 +10,6 @@
 	<xacro:property name="arm_length" value="0.124658905"/>
 	<xacro:property name="arm_width" value="0.1100"/>
-	<xacro:property name="arm_height" value="0.124658905"/>
+	<xacro:property name="arm_height" value="0.304997498"/>
+	<xacro:property name="arm_sphere_radius" value="0.03"/>
 	<xacro:property name="right_arm_center_of_mass" value="-0.001570 -0.001100 -0.074465"/>
 	<xacro:property name="left_arm_center_of_mass" value="-0.001570 0.001100 -0.074465"/>
@@ -67,4 +68,33 @@
 		<!-- transmission -->
 		<xacro:arm_transmission side="${side}"/>
+		<!-- arm sphere link -->
+		<link name="arm_sphere_${side}_link">
+			<collision>
+				<origin xyz="0 0 0" rpy="0 0 0"/>
+				<geometry>
+					<sphere radius="${arm_sphere_radius}"/>
+				</geometry>
+			</collision>
+			<visual>
+				<origin xyz="0 0 0" rpy="0 0 0"/>
+				<geometry>
+					<sphere radius="${arm_sphere_radius}"/>
+				</geometry>
+			</visual>
+			<inertial>
+				<origin xyz="0 0 0" rpy="0 0 0"/>
+				<inertia ixx="0.000001" ixy="0" ixz="0" iyy="0.000001" iyz="0" izz="0.000001"/>
+				<mass value="0.00001"/>
+			</inertial>
+		</link>
+		<gazebo reference="arm_sphere_${side}_link">
+			<material>Gazebo/Yellow</material>
+		</gazebo>
+		<!-- arm_sphere joint -->
+		<joint name="arm_sphere_${side}_joint" type="fixed">
+			<origin xyz="0 0 ${-arm_height + arm_sphere_radius + 0.02}" rpy="0 0 0"/>
+			<parent link="arm_${side}_link"/>
+			<child link="arm_sphere_${side}_link"/>
+		</joint>
 	</xacro:macro>
 	<!--***********************************************************************-->

File: stevie_description/urdf/head/head.xacro (robot description, xacro)
@@ -62,5 +62,5 @@
 				<origin xyz="0 0 0" rpy="0 ${PI/2} 0"/>
 				<mass value="0.00001"/>
-				<inertia ixx="1.0" ixy="0" ixz="0" iyy="1.0" iyz="0" izz="1.0"/>
+				<inertia ixx="0.000001" ixy="0" ixz="0" iyy="0.000001" iyz="0" izz="0.000001"/>
 			</inertial>
 		</link>
@@ -85,5 +85,5 @@
 				<origin xyz="0 0 0" rpy="0 ${PI/2} 0"/>
 				<mass value="0.00001"/>
-				<inertia ixx="1.0" ixy="0" ixz="0" iyy="1.0" iyz="0" izz="1.0"/>
+				<inertia ixx="0.000001" ixy="0" ixz="0" iyy="0.000001" iyz="0" izz="0.000001"/>
 			</inertial>
 		</link>
@@ -109,5 +109,5 @@
 				<origin xyz="0 0 0" rpy="0 ${PI/2} 0"/>
 				<mass value="0.00001"/>
-				<inertia ixx="1.0" ixy="0" ixz="0" iyy="1.0" iyz="0" izz="1.0"/>
+				<inertia ixx="0.000001" ixy="0" ixz="0" iyy="0.000001" iyz="0" izz="0.000001"/>
 			</inertial>
 		</link>

File: stevie_description/urdf/wheels/wheels.xacro (robot description, xacro)
@@ -71,5 +71,5 @@
 				<origin xyz="0 0 0" rpy="0 ${PI/2} 0"/>
 				<mass value="0.00001"/>
-				<inertia ixx="1.0" ixy="0" ixz="0" iyy="1.0" iyz="0" izz="1.0"/>
+				<inertia ixx="0.000001" ixy="0" ixz="0" iyy="0.000001" iyz="0" izz="0.000001"/>
 			</inertial>
 		</link>

Commit message: Navigation added. Still not tested

File: stevie_description/urdf/arms/arms.xacro (robot description, xacro)
@@ -24,5 +24,6 @@
 				<origin xyz="0 0 0" rpy="0 0 0"/>
 				<geometry>
-					<mesh filename="package://stevie_description/meshes/collision/${side}_arm_collision.stl" scale="0.001 0.001 0.001"/>
+					<!-- <mesh filename="package://stevie_description/meshes/collision/${side}_arm_collision.stl" scale="0.001 0.001 0.001"/> -->
+					<mesh filename="$(find stevie_description)/meshes/collision/${side}_arm_collision.stl" scale="0.001 0.001 0.001"/>
 				</geometry>
 			</collision>
@@ -30,5 +31,6 @@
 				<origin xyz="0 0 0" rpy="0 0 0"/>
 				<geometry>
-					<mesh filename="package://stevie_description/meshes/visual/${side}_arm.stl" scale="0.001 0.001 0.001"/>
+					<!-- <mesh filename="package://stevie_description/meshes/visual/${side}_arm.stl" scale="0.001 0.001 0.001"/> -->
+					<mesh filename="$(find stevie_description)/meshes/visual/${side}_arm.stl" scale="0.001 0.001 0.001"/>
 				</geometry>
 			</visual>

File: stevie_description/urdf/arms/shoulders.xacro (robot description, xacro)
@@ -19,5 +19,6 @@
 				<origin xyz="0 0 0" rpy="0 0 0"/>
 				<geometry>
-					<mesh filename="package://stevie_description/meshes/collision/shoulder_collision.stl" scale="0.001 0.001 0.001"/>
+					<!-- <mesh filename="package://stevie_description/meshes/collision/shoulder_collision.stl" scale="0.001 0.001 0.001"/> -->
+					<mesh filename="$(find stevie_description)/meshes/collision/shoulder_collision.stl" scale="0.001 0.001 0.001"/>
 				</geometry>
 			</collision>
@@ -25,5 +26,6 @@
 				<origin xyz="0 0 0" rpy="0 0 0"/>
 				<geometry>
-					<mesh filename="package://stevie_description/meshes/visual/shoulder.stl" scale="0.001 0.001 0.001"/>
+					<!-- <mesh filename="package://stevie_description/meshes/visual/shoulder.stl" scale="0.001 0.001 0.001"/> -->
+					<mesh filename="$(find stevie_description)/meshes/visual/shoulder.stl" scale="0.001 0.001 0.001"/>
 				</geometry>
 			</visual>

File: stevie_description/urdf/caster/caster.xacro (robot description, xacro)
@@ -23,5 +23,6 @@
 				<origin xyz="0 0 0" rpy="0 0 0"/>
 				<geometry>
-					<mesh filename="package://stevie_description/meshes/visual/caster.stl" scale="0.001 0.001 0.001"/>
+					<!-- <mesh filename="package://stevie_description/meshes/visual/caster.stl" scale="0.001 0.001 0.001"/> -->
+					<mesh filename="$(find stevie_description)/meshes/visual/caster.stl" scale="0.001 0.001 0.001"/>
 				</geometry>
 			</visual>

File: stevie_description/urdf/head/head.xacro (robot description, xacro)
@@ -18,5 +18,6 @@
 				<origin xyz="0 0 0" rpy="0 0 0"/>
 				<geometry>
-					<mesh filename="package://stevie_description/meshes/collision/head_collision.stl" scale="0.001 0.001 0.001"/>
+					<!-- <mesh filename="package://stevie_description/meshes/collision/head_collision.stl" scale="0.001 0.001 0.001"/> -->
+					<mesh filename="$(find stevie_description)/meshes/collision/head_collision.stl" scale="0.001 0.001 0.001"/>
 				</geometry>
 			</collision>
@@ -24,5 +25,6 @@
 				<origin xyz="0 0 0" rpy="0 0 0"/>
 				<geometry>
-			 		<mesh filename="package://stevie_description/meshes/visual/head.stl" scale="0.001 0.001 0.001"/>
+			 		<!-- <mesh filename="package://stevie_description/meshes/visual/head.stl" scale="0.001 0.001 0.001"/> -->
+			 		<mesh filename="$(find stevie_description)/meshes/visual/head.stl" scale="0.001 0.001 0.001"/>
 				</geometry>
 			</visual>
@@ -103,5 +105,6 @@
 				<origin xyz="0 0 0" rpy="0 0 0"/>
 				<geometry>
-					<mesh filename="package://stevie_description/meshes/visual/earcovers.stl" scale="0.001 0.001 0.001"/>
+					<!-- <mesh filename="package://stevie_description/meshes/visual/earcovers.stl" scale="0.001 0.001 0.001"/> -->
+					<mesh filename="$(find stevie_description)/meshes/visual/earcovers.stl" scale="0.001 0.001 0.001"/>
 				</geometry>
 			</visual>

File: stevie_description/urdf/head/neck.xacro (robot description, xacro)
@@ -21,5 +21,6 @@
 				<origin xyz="0 0 0" rpy="0 0 0"/>
 				<geometry>
-					<mesh filename="package://stevie_description/meshes/collision/neck_collision.stl" scale="0.001 0.001 0.001"/>
+					<!-- <mesh filename="package://stevie_description/meshes/collision/neck_collision.stl" scale="0.001 0.001 0.001"/> -->
+					<mesh filename="$(find stevie_description)/meshes/collision/neck_collision.stl" scale="0.001 0.001 0.001"/>
 				</geometry>
 			</collision>
@@ -27,5 +28,6 @@
 				<origin xyz="0 0 0" rpy="0 0 0"/>
 					<geometry>
-				 		<mesh filename="package://stevie_description/meshes/visual/neck.stl" scale="0.001 0.001 0.001"/>
+				 		<!-- <mesh filename="package://stevie_description/meshes/visual/neck.stl" scale="0.001 0.001 0.001"/> -->
+				 		<mesh filename="$(find stevie_description)/meshes/visual/neck.stl" scale="0.001 0.001 0.001"/>
 					</geometry>
 			</visual>

File: stevie_description/urdf/lower_body/lower_body.xacro (robot description, xacro)
@@ -24,5 +24,6 @@
 				<origin xyz="0 0 0" rpy="0 0 0"/>
 				<geometry>
-					<mesh filename="package://stevie_description/meshes/collision/lower_body_collision.stl" scale="0.001 0.001 0.001"/>
+					<!-- <mesh filename="package://stevie_description/meshes/collision/lower_body_collision.stl" scale="0.001 0.001 0.001"/> -->
+					<mesh filename="$(find stevie_description)/meshes/collision/lower_body_collision.stl" scale="0.001 0.001 0.001"/>
 				</geometry>
 			</collision>
@@ -30,5 +31,6 @@
 				<origin xyz="0 0 0" rpy="0 0 0"/>
 					<geometry>
-				 		<mesh filename="package://stevie_description/meshes/visual/lower_body.stl" scale="0.001 0.001 0.001"/>
+				 		<!-- <mesh filename="package://stevie_description/meshes/visual/lower_body.stl" scale="0.001 0.001 0.001"/> -->
+				 		<mesh filename="$(find stevie_description)/meshes/visual/lower_body.stl" scale="0.001 0.001 0.001"/>
 					</geometry>
 			</visual>

File: stevie_description/urdf/upper_body/hip.xacro (robot description, xacro)
@@ -19,5 +19,6 @@
 				<origin xyz="0 0 0" rpy="0 0 0"/>
 				<geometry>
-					<mesh filename="package://stevie_description/meshes/collision/hip_upper_collision.stl" scale="0.001 0.001 0.001"/>
+					<!-- <mesh filename="package://stevie_description/meshes/collision/hip_upper_collision.stl" scale="0.001 0.001 0.001"/> -->
+					<mesh filename="$(find stevie_description)/meshes/collision/hip_upper_collision.stl" scale="0.001 0.001 0.001"/>
 				</geometry>
 			</collision>
@@ -25,5 +26,6 @@
 				<origin xyz="0 0 0" rpy="0 0 0"/>
 				<geometry>
-			 		<mesh filename="package://stevie_description/meshes/visual/hip_upper.stl" scale="0.001 0.001 0.001"/>
+			 		<!-- <mesh filename="package://stevie_description/meshes/visual/hip_upper.stl" scale="0.001 0.001 0.001"/> -->
+			 		<mesh filename="$(find stevie_description)/meshes/visual/hip_upper.stl" scale="0.001 0.001 0.001"/>
 				</geometry>
 			</visual>

File: stevie_description/urdf/upper_body/upper_body.xacro (robot description, xacro)
@@ -1,5 +1,5 @@
 <?xml version="1.0"?>
 <robot  xmlns:xacro="http://ros.org/wiki/xacro">
-	<xacro:include filename="$(find stevie_description)/urdf/upper_body/upper_body.transmission.xacro" />
+	<!-- <xacro:include filename="$(find stevie_description)/urdf/upper_body/upper_body.transmission.xacro" /> -->
 	<xacro:include filename="$(find stevie_description)/urdf/upper_body/hip.xacro" />
 	<!-- DECLARE VARIABLES -->
@@ -18,5 +18,6 @@
 				<origin xyz="0 0 0" rpy="0 0 0"/>
 				<geometry>
-					<mesh filename="package://stevie_description/meshes/collision/upper_body_collision.stl" scale="0.001 0.001 0.001"/>
+					<!-- <mesh filename="package://stevie_description/meshes/collision/upper_body_collision.stl" scale="0.001 0.001 0.001"/> -->
+					<mesh filename="$(find stevie_description)/meshes/collision/upper_body_collision.stl" scale="0.001 0.001 0.001"/>
 				</geometry>
 			</collision>
@@ -24,5 +25,6 @@
 				<origin xyz="0 0 0" rpy="0 0 0"/>
 				<geometry>
-			 		<mesh filename="package://stevie_description/meshes/visual/upper_body.stl" scale="0.001 0.001 0.001"/>
+			 		<!-- <mesh filename="package://stevie_description/meshes/visual/upper_body.stl" scale="0.001 0.001 0.001"/> -->
+			 		<mesh filename="$(find stevie_description)/meshes/visual/upper_body.stl" scale="0.001 0.001 0.001"/>
 				</geometry>
 			</visual>

File: stevie_description/urdf/wheels/wheels.xacro (robot description, xacro)
@@ -23,5 +23,6 @@
 				<origin xyz="0 0 0" rpy="0 0 0"/>
 				<geometry>
-					<mesh filename="package://stevie_description/meshes/visual/wheel.stl" scale="0.001 0.001 0.001"/>
+					<!-- <mesh filename="package://stevie_description/meshes/visual/wheel.stl" scale="0.001 0.001 0.001"/> -->
+					<mesh filename="$(find stevie_description)/meshes/visual/wheel.stl" scale="0.001 0.001 0.001"/>
 				</geometry>
 			</visual>
@@ -33,6 +34,6 @@
 		</link>
 		<gazebo reference="wheel_${side}_link">
-			<mu1>1.0</mu1>
-			<mu2>1.0</mu2>
+			<mu1>100.0</mu1>
+			<mu2>50.0</mu2>
 			<!--kp value="10000000.0"/>
       <kd value="100.0"/>
@@ -65,5 +66,6 @@
 				<geometry>
 					<!-- slightly larger scale so the yellow cap can cover the one already on the wheel mesh -->
-					<mesh filename="package://stevie_description/meshes/visual/wheel_cap.stl" scale="0.001001 0.001001 0.001001"/>
+					<!-- <mesh filename="package://stevie_description/meshes/visual/wheel_cap.stl" scale="0.001001 0.001001 0.001001"/> -->
+					<mesh filename="$(find stevie_description)/meshes/visual/wheel_cap.stl" scale="0.001001 0.001001 0.001001"/>
 				</geometry>
 			</visual>
