Commit message: Ajout d'un launchfile affichant les capteurs de Stevie

File: stevie_description/urdf/arms/arms.xacro (robot description, xacro)
@@ -24,6 +24,6 @@
 				<origin xyz="0 0 0" rpy="0 0 0"/>
 				<geometry>
-					<!-- <mesh filename="package://stevie_description/meshes/collision/${side}_arm_collision.stl" scale="0.001 0.001 0.001"/> -->
-					<mesh filename="$(find stevie_description)/meshes/collision/${side}_arm_collision.stl" scale="0.001 0.001 0.001"/>
+					<mesh filename="package://stevie_description/meshes/collision/${side}_arm_collision.stl" scale="0.001 0.001 0.001"/>
+					<!-- <mesh filename="$(find stevie_description)/meshes/collision/${side}_arm_collision.stl" scale="0.001 0.001 0.001"/> -->
 				</geometry>
 			</collision>
@@ -31,6 +31,6 @@
 				<origin xyz="0 0 0" rpy="0 0 0"/>
 				<geometry>
-					<!-- <mesh filename="package://stevie_description/meshes/visual/${side}_arm.stl" scale="0.001 0.001 0.001"/> -->
-					<mesh filename="$(find stevie_description)/meshes/visual/${side}_arm.stl" scale="0.001 0.001 0.001"/>
+					<mesh filename="package://stevie_description/meshes/visual/${side}_arm.stl" scale="0.001 0.001 0.001"/>
+					<!-- <mesh filename="$(find stevie_description)/meshes/visual/${side}_arm.stl" scale="0.001 0.001 0.001"/> -->
 				</geometry>
 			</visual>

File: stevie_description/urdf/arms/shoulders.xacro (robot description, xacro)
@@ -19,6 +19,6 @@
 				<origin xyz="0 0 0" rpy="0 0 0"/>
 				<geometry>
-					<!-- <mesh filename="package://stevie_description/meshes/collision/shoulder_collision.stl" scale="0.001 0.001 0.001"/> -->
-					<mesh filename="$(find stevie_description)/meshes/collision/shoulder_collision.stl" scale="0.001 0.001 0.001"/>
+					<mesh filename="package://stevie_description/meshes/collision/shoulder_collision.stl" scale="0.001 0.001 0.001"/>
+					<!-- <mesh filename="$(find stevie_description)/meshes/collision/shoulder_collision.stl" scale="0.001 0.001 0.001"/> -->
 				</geometry>
 			</collision>
@@ -26,6 +26,6 @@
 				<origin xyz="0 0 0" rpy="0 0 0"/>
 				<geometry>
-					<!-- <mesh filename="package://stevie_description/meshes/visual/shoulder.stl" scale="0.001 0.001 0.001"/> -->
-					<mesh filename="$(find stevie_description)/meshes/visual/shoulder.stl" scale="0.001 0.001 0.001"/>
+					<mesh filename="package://stevie_description/meshes/visual/shoulder.stl" scale="0.001 0.001 0.001"/>
+					<!-- <mesh filename="$(find stevie_description)/meshes/visual/shoulder.stl" scale="0.001 0.001 0.001"/> -->
 				</geometry>
 			</visual>

File: stevie_description/urdf/caster/caster.xacro (robot description, xacro)
@@ -23,6 +23,6 @@
 				<origin xyz="0 0 0" rpy="0 0 0"/>
 				<geometry>
-					<!-- <mesh filename="package://stevie_description/meshes/visual/caster.stl" scale="0.001 0.001 0.001"/> -->
-					<mesh filename="$(find stevie_description)/meshes/visual/caster.stl" scale="0.001 0.001 0.001"/>
+					<mesh filename="package://stevie_description/meshes/visual/caster.stl" scale="0.001 0.001 0.001"/>
+					<!-- <mesh filename="$(find stevie_description)/meshes/visual/caster.stl" scale="0.001 0.001 0.001"/> -->
 				</geometry>
 			</visual>

File: stevie_description/urdf/head/head.xacro (robot description, xacro)
@@ -18,6 +18,6 @@
 				<origin xyz="0 0 0" rpy="0 0 0"/>
 				<geometry>
-					<!-- <mesh filename="package://stevie_description/meshes/collision/head_collision.stl" scale="0.001 0.001 0.001"/> -->
-					<mesh filename="$(find stevie_description)/meshes/collision/head_collision.stl" scale="0.001 0.001 0.001"/>
+					<mesh filename="package://stevie_description/meshes/collision/head_collision.stl" scale="0.001 0.001 0.001"/>
+					<!-- <mesh filename="$(find stevie_description)/meshes/collision/head_collision.stl" scale="0.001 0.001 0.001"/> -->
 				</geometry>
 			</collision>
@@ -25,6 +25,6 @@
 				<origin xyz="0 0 0" rpy="0 0 0"/>
 				<geometry>
-			 		<!-- <mesh filename="package://stevie_description/meshes/visual/head.stl" scale="0.001 0.001 0.001"/> -->
-			 		<mesh filename="$(find stevie_description)/meshes/visual/head.stl" scale="0.001 0.001 0.001"/>
+			 		<mesh filename="package://stevie_description/meshes/visual/head.stl" scale="0.001 0.001 0.001"/>
+			 		<!-- <mesh filename="$(find stevie_description)/meshes/visual/head.stl" scale="0.001 0.001 0.001"/> -->
 				</geometry>
 			</visual>
@@ -105,6 +105,6 @@
 				<origin xyz="0 0 0" rpy="0 0 0"/>
 				<geometry>
-					<!-- <mesh filename="package://stevie_description/meshes/visual/earcovers.stl" scale="0.001 0.001 0.001"/> -->
-					<mesh filename="$(find stevie_description)/meshes/visual/earcovers.stl" scale="0.001 0.001 0.001"/>
+					<mesh filename="package://stevie_description/meshes/visual/earcovers.stl" scale="0.001 0.001 0.001"/>
+					<!-- <mesh filename="$(find stevie_description)/meshes/visual/earcovers.stl" scale="0.001 0.001 0.001"/> -->
 				</geometry>
 			</visual>

File: stevie_description/urdf/head/neck.xacro (robot description, xacro)
@@ -21,6 +21,6 @@
 				<origin xyz="0 0 0" rpy="0 0 0"/>
 				<geometry>
-					<!-- <mesh filename="package://stevie_description/meshes/collision/neck_collision.stl" scale="0.001 0.001 0.001"/> -->
-					<mesh filename="$(find stevie_description)/meshes/collision/neck_collision.stl" scale="0.001 0.001 0.001"/>
+					<mesh filename="package://stevie_description/meshes/collision/neck_collision.stl" scale="0.001 0.001 0.001"/>
+					<!-- <mesh filename="$(find stevie_description)/meshes/collision/neck_collision.stl" scale="0.001 0.001 0.001"/> -->
 				</geometry>
 			</collision>
@@ -28,6 +28,6 @@
 				<origin xyz="0 0 0" rpy="0 0 0"/>
 					<geometry>
-				 		<!-- <mesh filename="package://stevie_description/meshes/visual/neck.stl" scale="0.001 0.001 0.001"/> -->
-				 		<mesh filename="$(find stevie_description)/meshes/visual/neck.stl" scale="0.001 0.001 0.001"/>
+				 		<mesh filename="package://stevie_description/meshes/visual/neck.stl" scale="0.001 0.001 0.001"/>
+				 		<!-- <mesh filename="$(find stevie_description)/meshes/visual/neck.stl" scale="0.001 0.001 0.001"/> -->
 					</geometry>
 			</visual>

File: stevie_description/urdf/lower_body/lower_body.xacro (robot description, xacro)
@@ -24,6 +24,6 @@
 				<origin xyz="0 0 0" rpy="0 0 0"/>
 				<geometry>
-					<!-- <mesh filename="package://stevie_description/meshes/collision/lower_body_collision.stl" scale="0.001 0.001 0.001"/> -->
-					<mesh filename="$(find stevie_description)/meshes/collision/lower_body_collision.stl" scale="0.001 0.001 0.001"/>
+					<mesh filename="package://stevie_description/meshes/collision/lower_body_collision.stl" scale="0.001 0.001 0.001"/>
+					<!-- <mesh filename="$(find stevie_description)/meshes/collision/lower_body_collision.stl" scale="0.001 0.001 0.001"/> -->
 				</geometry>
 			</collision>
@@ -31,6 +31,6 @@
 				<origin xyz="0 0 0" rpy="0 0 0"/>
 					<geometry>
-				 		<!-- <mesh filename="package://stevie_description/meshes/visual/lower_body.stl" scale="0.001 0.001 0.001"/> -->
-				 		<mesh filename="$(find stevie_description)/meshes/visual/lower_body.stl" scale="0.001 0.001 0.001"/>
+				 		<mesh filename="package://stevie_description/meshes/visual/lower_body.stl" scale="0.001 0.001 0.001"/>
+				 		<!-- <mesh filename="$(find stevie_description)/meshes/visual/lower_body.stl" scale="0.001 0.001 0.001"/> -->
 					</geometry>
 			</visual>

File: stevie_description/urdf/upper_body/hip.xacro (robot description, xacro)
@@ -19,6 +19,6 @@
 				<origin xyz="0 0 0" rpy="0 0 0"/>
 				<geometry>
-					<!-- <mesh filename="package://stevie_description/meshes/collision/hip_upper_collision.stl" scale="0.001 0.001 0.001"/> -->
-					<mesh filename="$(find stevie_description)/meshes/collision/hip_upper_collision.stl" scale="0.001 0.001 0.001"/>
+					<mesh filename="package://stevie_description/meshes/collision/hip_upper_collision.stl" scale="0.001 0.001 0.001"/>
+					<!-- <mesh filename="$(find stevie_description)/meshes/collision/hip_upper_collision.stl" scale="0.001 0.001 0.001"/> -->
 				</geometry>
 			</collision>
@@ -26,6 +26,6 @@
 				<origin xyz="0 0 0" rpy="0 0 0"/>
 				<geometry>
-			 		<!-- <mesh filename="package://stevie_description/meshes/visual/hip_upper.stl" scale="0.001 0.001 0.001"/> -->
-			 		<mesh filename="$(find stevie_description)/meshes/visual/hip_upper.stl" scale="0.001 0.001 0.001"/>
+			 		<mesh filename="package://stevie_description/meshes/visual/hip_upper.stl" scale="0.001 0.001 0.001"/>
+			 		<!-- <mesh filename="$(find stevie_description)/meshes/visual/hip_upper.stl" scale="0.001 0.001 0.001"/> -->
 				</geometry>
 			</visual>

File: stevie_description/urdf/upper_body/upper_body.xacro (robot description, xacro)
@@ -18,6 +18,6 @@
 				<origin xyz="0 0 0" rpy="0 0 0"/>
 				<geometry>
-					<!-- <mesh filename="package://stevie_description/meshes/collision/upper_body_collision.stl" scale="0.001 0.001 0.001"/> -->
-					<mesh filename="$(find stevie_description)/meshes/collision/upper_body_collision.stl" scale="0.001 0.001 0.001"/>
+					<mesh filename="package://stevie_description/meshes/collision/upper_body_collision.stl" scale="0.001 0.001 0.001"/>
+					<!-- <mesh filename="$(find stevie_description)/meshes/collision/upper_body_collision.stl" scale="0.001 0.001 0.001"/> -->
 				</geometry>
 			</collision>
@@ -25,6 +25,6 @@
 				<origin xyz="0 0 0" rpy="0 0 0"/>
 				<geometry>
-			 		<!-- <mesh filename="package://stevie_description/meshes/visual/upper_body.stl" scale="0.001 0.001 0.001"/> -->
-			 		<mesh filename="$(find stevie_description)/meshes/visual/upper_body.stl" scale="0.001 0.001 0.001"/>
+			 		<mesh filename="package://stevie_description/meshes/visual/upper_body.stl" scale="0.001 0.001 0.001"/>
+			 		<!-- <mesh filename="$(find stevie_description)/meshes/visual/upper_body.stl" scale="0.001 0.001 0.001"/> -->
 				</geometry>
 			</visual>

File: stevie_description/urdf/wheels/wheels.xacro (robot description, xacro)
@@ -23,6 +23,6 @@
 				<origin xyz="0 0 0" rpy="0 0 0"/>
 				<geometry>
-					<!-- <mesh filename="package://stevie_description/meshes/visual/wheel.stl" scale="0.001 0.001 0.001"/> -->
-					<mesh filename="$(find stevie_description)/meshes/visual/wheel.stl" scale="0.001 0.001 0.001"/>
+					<mesh filename="package://stevie_description/meshes/visual/wheel.stl" scale="0.001 0.001 0.001"/>
+					<!-- <mesh filename="$(find stevie_description)/meshes/visual/wheel.stl" scale="0.001 0.001 0.001"/> -->
 				</geometry>
 			</visual>
@@ -66,6 +66,6 @@
 				<geometry>
 					<!-- slightly larger scale so the yellow cap can cover the one already on the wheel mesh -->
-					<!-- <mesh filename="package://stevie_description/meshes/visual/wheel_cap.stl" scale="0.001001 0.001001 0.001001"/> -->
-					<mesh filename="$(find stevie_description)/meshes/visual/wheel_cap.stl" scale="0.001001 0.001001 0.001001"/>
+					<mesh filename="package://stevie_description/meshes/visual/wheel_cap.stl" scale="0.001001 0.001001 0.001001"/>
+					<!-- <mesh filename="$(find stevie_description)/meshes/visual/wheel_cap.stl" scale="0.001001 0.001001 0.001001"/> -->
 				</geometry>
 			</visual>
