Commit message: Hip added

File: stevie_description/urdf/caster/caster.xacro (robot description, xacro)
@@ -11,10 +11,10 @@
 	<xacro:property name="PI" value="3.14159"/>
 	<!--**************   MOMENT OF INERTIA OF A SPHERE   **************-->
-	<macro name="sphere_inertia" params="m r">
+	<xacro:macro name="sphere_inertia" params="m r">
     <inertia  ixx="${2*m*r*r/5}" ixy="0" ixz="0"
               iyy="${2*m*r*r/5}" iyz="0"
               izz="${2*m*r*r/5}"
     />
-  </macro>
+  </xacro:macro>
 	<!--***************************************************************-->
 	<!--************************        CASTER          ************************-->

File: stevie_description/urdf/stevie.xacro (robot description, xacro)
@@ -23,4 +23,6 @@
 -->
   <xacro:include filename="$(find stevie_description)/urdf/lower_body/lower_body.xacro" />
+  <xacro:include filename="$(find stevie_description)/urdf/upper_body/hip.xacro" />
   <xacro:lower_body  name="lower_body"/>
+  <xacro:hip parent="lower_body_link"/>
 </robot>

Commit message: Caster radius corrected + simplified inertia for the wheels and the caster

File: stevie_description/urdf/caster/caster.xacro (robot description, xacro)
@@ -6,5 +6,5 @@
 	<!-- DECLARE VARIABLES -->
 	<xacro:property name="caster_mass" value="0.5"/>
-	<xacro:property name="caster_radius" value="0.133"/>
+	<xacro:property name="caster_radius" value="0.05"/>
 	<xacro:property name="caster_x_adjustment" value="-0.3055"/>
 	<xacro:property name="caster_z_adjustment" value="-0.05"/>
@@ -25,5 +25,5 @@
 				<origin xyz="0 0 0" rpy="0 0 0"/>
 				<geometry>
-					<mesh filename="package://stevie_description/meshes/collision/caster_collision.STL" scale="0.001 0.001 0.001"/>
+					<sphere radius="${caster_radius}"/>
 				</geometry>
 			</collision>
@@ -31,5 +31,5 @@
 				<origin xyz="0 0 0" rpy="0 0 0"/>
 				<geometry>
-					<mesh filename="package://stevie_description/meshes/visual/caster.STL" scale="0.001 0.001 0.001"/>
+					<mesh filename="package://stevie_description/meshes/collision/caster_collision.STL" scale="0.001 0.001 0.001"/>
 				</geometry>
 			</visual>

File: stevie_description/urdf/wheels/wheels.xacro (robot description, xacro)
@@ -21,7 +21,7 @@
 		<link name="wheel_${side}_link">
 			<collision>
-				<origin xyz="0 0 0" rpy="0 0 0"/>
+				<origin xyz="0 0 0" rpy="0 ${PI/2} 0"/>
 				<geometry>
-					<mesh filename="package://stevie_description/meshes/collision/wheel_collision.STL" scale="0.001 0.001 0.001"/>
+			 		<cylinder length="${wheel_thickness}" radius="${wheel_radius}"/>
 				</geometry>
 			</collision>
@@ -29,5 +29,5 @@
 				<origin xyz="0 0 0" rpy="0 0 0"/>
 				<geometry>
-			 		<mesh filename="package://stevie_description/meshes/visual/wheel.STL" scale="0.001 0.001 0.001"/>
+					<mesh filename="package://stevie_description/meshes/collision/wheel_collision.STL" scale="0.001 0.001 0.001"/>
 				</geometry>
 			</visual>

Commit message: Lasers and cameras working + diff_drive_controller working (but robot slow)

File: stevie_description/urdf/caster/caster.xacro (robot description, xacro)
@@ -6,5 +6,5 @@
 	<!-- DECLARE VARIABLES -->
 	<xacro:property name="caster_mass" value="0.5"/>
-	<xacro:property name="caster_radius" value="0.05"/>
+	<xacro:property name="caster_radius" value="0.052"/>
 	<xacro:property name="caster_x_adjustment" value="-0.3055"/>
 	<xacro:property name="caster_z_adjustment" value="-0.05"/>

File: stevie_description/urdf/head/head.xacro (robot description, xacro)
@@ -9,10 +9,4 @@
 	<xacro:property name="head_height" value="0.300608185"/>
 	<xacro:property name="PI" value="3.14159"/>
-	<xacro:macro name="box_inertia" params="m x y z">
-    <inertia  ixx="${m*(y*y+z*z)/12}" ixy="0" ixz="0"
-              iyy="${m*(x*x+z*z)/12}" iyz="0"
-              izz="${m*(x*x+z*z)/12}"
-    />
-  </xacro:macro>
 	<!--************************        HEAD          ************************-->
   <xacro:macro name="head" params="parent" >

File: stevie_description/urdf/stevie.xacro (robot description, xacro)
@@ -1,13 +1,25 @@
 <?xml version="1.0"?>
 <robot name="stevie" xmlns:xacro="http://ros.org/wiki/xacro">
-  <xacro:include filename="$(find stevie_description)/urdf/macro.xacro" />
-  <xacro:include filename="$(find stevie_description)/urdf/stevie.gazebo"/>
-  <!-- LOAD ROBOT COMPONENT FILES -->
+  <!-- VARIABLES -->
   <xacro:property name="lower_body_name" value="lower_body"/>
   <xacro:property name="upper_body_name" value="upper_body"/>
+	<xacro:property name="front_left_camera_name" value="front_left_camera"/>
+	<xacro:property name="front_right_camera_name" value="front_right_camera"/>
+	<xacro:property name="back_camera_name" value="back_camera"/>
+	<xacro:property name="top_camera_name" value="top_camera"/>
+	<xacro:property name="front_laser_name" value="front_laser"/>
+	<xacro:property name="back_laser_name" value="back_laser"/>
+	<xacro:property name="kinect_name" value="kinect"/>
+	<xacro:property name="PI" value="3.14159"/>
+  <!-- DEPENDENCIES -->
+  <xacro:include filename="$(find stevie_description)/urdf/macros.xacro" />
+  <xacro:include filename="$(find stevie_description)/urdf/stevie.gazebo"/>
+  <xacro:include filename="$(find stevie_description)/urdf/sensors/sensor_macros.xacro"/>
+  <!-- LOAD ROBOT COMPONENT FILES -->
   <xacro:include filename="$(find stevie_description)/urdf/lower_body/lower_body.xacro" />
   <xacro:include filename="$(find stevie_description)/urdf/upper_body/upper_body.xacro" />
   <xacro:include filename="$(find stevie_description)/urdf/arms/arms.xacro" />
   <xacro:include filename="$(find stevie_description)/urdf/head/head.xacro" />
+  <!-- ROBOT COMPONENTS -->
   <xacro:lower_body  name="${lower_body_name}"/>
   <xacro:upper_body parent="${lower_body_name}_link" name="${upper_body_name}"/>
@@ -15,3 +27,14 @@
   <xacro:arm parent="${upper_body_name}_link" side="right"/>
   <xacro:head parent="${upper_body_name}_link"/>
+  <!-- SENSORS -->
+  <!-- cameras -->
+	<xacro:camera name="${front_left_camera_name}" parent="${upper_body_name}_link" xyz="0.11 -0.09 0.49" rpy="0 0 0"/>
+	<xacro:camera name="${front_right_camera_name}" parent="${upper_body_name}_link" xyz="0.11 0.09 0.49" rpy="0 0 0"/>
+	<xacro:camera name="${back_camera_name}" parent="${upper_body_name}_link" xyz="-0.12 0 0.49" rpy="0 0 ${PI}"/>
+	<xacro:camera name="${top_camera_name}" parent="head_link" xyz="0.02 0 0.28" rpy="0 0 0"/>
+  <!-- Hokuyo lasers -->
+	<xacro:laser name="${front_laser_name}" parent="${lower_body_name}_link" xyz="0.003 0 0.358" rpy="0 0 0"/>
+	<xacro:laser name="${back_laser_name}" parent="${lower_body_name}_link" xyz="-0.275 0 0.358" rpy="0 0 ${PI}"/>
+	<!-- Kinect camera -->
+	<xacro:kinect name="${kinect_name}" parent="${upper_body_name}_link" xyz="0.14 0 0.4" rpy="0 0 0"/>
 </robot>

File: stevie_description/urdf/upper_body/hip.xacro (robot description, xacro)
@@ -10,5 +10,5 @@
 	<xacro:property name="hip_center_of_mass" value="0 0 -0.056289"/>
 	<xacro:property name="hip_x_adjustment" value="-0.135"/>
-	<xacro:property name="hip_z_adjustment" value="0.43"/>
+	<xacro:property name="hip_z_adjustment" value="0.44"/>
 	<xacro:property name="PI" value="3.14159"/>
 	<!--************************        HIP          ************************-->
@@ -41,5 +41,5 @@
 		</gazebo>
 		<!-- lower_body-hip joint -->
-		<joint name="hip_lower_body_joint" type="revolute">
+		<joint name="lower_body_hip_joint" type="revolute">
 			<origin xyz="${hip_x_adjustment} 0 ${hip_z_adjustment}" rpy="0 0 0"/>
 			<axis xyz="0 0 1"/>

File: stevie_description/urdf/upper_body/upper_body.transmission.xacro (robot description, xacro)
@@ -5,5 +5,5 @@
 		<transmission name="hip_transmission">
 			<type>transmission_interface/SimpleTransmission</type>
-			<joint name="hip_lower_body_joint">
+			<joint name="lower_body_hip_joint">
 				<hardwareInterface>hardware_interface/EffortJointInterface</hardwareInterface>
     		</joint>
@@ -18,5 +18,5 @@
 		<transmission name="upper_body_transmission">
 			<type>transmission_interface/SimpleTransmission</type>
-			<joint name="upper_body_hip_joint">
+			<joint name="hip_upper_body_joint">
 				<hardwareInterface>hardware_interface/EffortJointInterface</hardwareInterface>
     		</joint>

File: stevie_description/urdf/upper_body/upper_body.xacro (robot description, xacro)
@@ -42,5 +42,5 @@
 		<xacro:hip parent="${parent}"/>
 		<!-- upper_body-hip joint -->
-		<joint name="upper_body_hip_joint" type="revolute">
+		<joint name="hip_upper_body_joint" type="revolute">
 			<origin xyz="0 0 0" rpy="0 0 0"/>
 			<axis xyz="0 1 0"/>

File: stevie_description/urdf/wheels/wheels.transmission.xacro (robot description, xacro)
@@ -5,8 +5,8 @@
 			<type>transmission_interface/SimpleTransmission</type>
 			<joint name="wheel_${side}_joint">
-				<hardwareInterface>hardware_interface/EffortJointInterface</hardwareInterface>
+				<hardwareInterface>hardware_interface/VelocityJointInterface</hardwareInterface>
     		</joint>
 			<actuator name="${side}_motor">
-				<hardwareInterface>hardware_interface/EffortJointInterface</hardwareInterface>
+				<hardwareInterface>hardware_interface/VelocityJointInterface</hardwareInterface>
 				<mechanicalReduction>1</mechanicalReduction>
 			</actuator>

File: stevie_description/urdf/wheels/wheels.xacro (robot description, xacro)
@@ -10,10 +10,4 @@
 	<xacro:property name="chassis_width" value="0.5"/>
 	<xacro:property name="PI" value="3.14159"/>
-	<xacro:macro name="cylinder_inertia" params="m r h">
-	  <inertia  ixx="${m*(3*r*r+h*h)/12}" ixy = "0" ixz = "0"
-	    iyy="${m*(3*r*r+h*h)/12}" iyz = "0"
-	    izz="${m*r*r/2}"
-	  />
-	</xacro:macro>
 	<!--************************        WHEELS          ************************-->
   <xacro:macro name="wheel" params="parent side" >

Commit message: Changed the collision file names from .STL to .stl + added the eyes and the mouth on stevie's head

File: stevie_description/urdf/caster/caster.xacro (robot description, xacro)
@@ -10,12 +10,4 @@
 	<xacro:property name="caster_z_adjustment" value="-0.05"/>
 	<xacro:property name="PI" value="3.14159"/>
-	<!--**************   MOMENT OF INERTIA OF A SPHERE   **************-->
-	<xacro:macro name="sphere_inertia" params="m r">
-    <inertia  ixx="${2*m*r*r/5}" ixy="0" ixz="0"
-              iyy="${2*m*r*r/5}" iyz="0"
-              izz="${2*m*r*r/5}"
-    />
-  </xacro:macro>
-	<!--***************************************************************-->
 	<!--************************        CASTER          ************************-->
   <xacro:macro name="caster" params="parent" >
@@ -43,5 +35,4 @@
 			<mu1>0.0</mu1>
 			<mu2>0.0</mu2>
-			<maxVel>0</maxVel>
 			<material>Gazebo/Black</material>
 		</gazebo>

File: stevie_description/urdf/head/head.xacro (robot description, xacro)
@@ -23,12 +23,12 @@
 			<visual>
 				<origin xyz="0 0 0" rpy="0 0 0"/>
-					<geometry>
-				 		<mesh filename="package://stevie_description/meshes/visual/head.stl" scale="0.001 0.001 0.001"/>
-					</geometry>
+				<geometry>
+			 		<mesh filename="package://stevie_description/meshes/visual/head.stl" scale="0.001 0.001 0.001"/>
+				</geometry>
 			</visual>
 			<inertial>
 				<origin xyz="0 0 ${head_height / 2}" rpy="0 0 0"/>
 				<mass value="${head_mass}"/>
-				<xacro:box_inertia m="${head_mass}" x="${head_width}" y="${head_height}" z="${head_length}"/>
+				<xacro:box_inertia m="${head_mass}" x="${head_width}" y="${head_length}" z="${head_height}"/>
 			</inertial>
 		</link>
@@ -56,5 +56,5 @@
 				<origin xyz="0 0 0" rpy="0 0 0"/>
 				<geometry>
-					<mesh filename="package://stevie_description/meshes/visual/upper_screen.stl" scale="0.001001 0.001001 0.001001"/>
+					<box size="0.001 0.18 0.14"/>
 				</geometry>
 			</visual>
@@ -66,9 +66,9 @@
 		</link>
 		<gazebo reference="upper_screen_link">
-			<material>Gazebo/Black</material>
+			<xacro:eyes/>
 		</gazebo>
 		<!-- upper_screen joint -->
 		<joint name="upper_screen_joint" type="fixed">
-			<origin xyz="0 0 0" rpy="0 0 0"/>
+			<origin xyz="0.11128992 0 0.18088210" rpy="0 -0.31 0"/>
 			<parent link="head_link"/>
 			<child link="upper_screen_link"/>
@@ -79,5 +79,5 @@
 				<origin xyz="0 0 0" rpy="0 0 0"/>
 				<geometry>
-					<mesh filename="package://stevie_description/meshes/visual/lower_screen.stl" scale="0.001001 0.001001 0.001001"/>
+					<box size="0.001 0.14 0.11"/>
 				</geometry>
 			</visual>
@@ -89,9 +89,9 @@
 		</link>
 		<gazebo reference="lower_screen_link">
-			<material>Gazebo/Black</material>
+			<xacro:mouth/>
 		</gazebo>
 		<!-- lower_screen joint -->
 		<joint name="lower_screen_joint" type="fixed">
-			<origin xyz="0 0 0" rpy="0 0 0"/>
+			<origin xyz="0.11499191 0 0.04708293" rpy="0 0.3 0"/>
 			<parent link="head_link"/>
 			<child link="lower_screen_link"/>

File: stevie_description/urdf/lower_body/lower_body.xacro (robot description, xacro)
@@ -7,15 +7,16 @@
 	<xacro:include filename="$(find stevie_description)/urdf/caster/caster.xacro" />
 	<!-- DECLARE VARIABLES -->
-	<xacro:property name="lower_body_mass" value="27"/>
+	<xacro:property name="lower_body_mass" value="40"/>
 	<xacro:property name="lower_body_volume" value="0.016607"/>
 	<xacro:property name="lower_body_length" value="0.485903"/>
 	<xacro:property name="lower_body_width" value="0.516555"/>
 	<xacro:property name="lower_body_height" value="0.475"/>
-	<xacro:property name="lower_body_center_of_mass" value="-0.112043 0.000001 0.051805"/>
+	<!--xacro:property name="lower_body_center_of_mass" value="-0.112043 0.000001 0.051805"/-->
+	<xacro:property name="lower_body_center_of_mass" value="-0.212043 0.000001 0"/>
 	<xacro:property name="PI" value="3.14159"/>
 	<!--************************        LOWER BODY          ************************-->
   <xacro:macro name="lower_body" params="name" >
 		<!-- base link -->
-		<link name="${name}_footprint" />
+		<link name="${name}_footprint"/>
 		<!-- lower body link -->
 		<link name="${name}_link">

File: stevie_description/urdf/macros.xacro (robot description, xacro)
@@ -12,5 +12,12 @@
     <inertia  ixx="${m*(y*y+z*z)/12}" ixy="0" ixz="0"
               iyy="${m*(x*x+z*z)/12}" iyz="0"
-              izz="${m*(x*x+z*z)/12}"
+              izz="${m*(x*x+y*y)/12}"
+    />
+  </xacro:macro>
+  <!-- compute the inertia of a sphere -->
+  <xacro:macro name="sphere_inertia" params="m r">
+    <inertia  ixx="${2*m*r*r/5}" ixy="0" ixz="0"
+              iyy="${2*m*r*r/5}" iyz="0"
+              izz="${2*m*r*r/5}"
     />
   </xacro:macro>
@@ -22,3 +29,17 @@
 	  />
 	</xacro:macro>
+  <!-- creates a counterweight to move the center of mass of a link -->
+	<xacro:macro name="counterweight" params="parent m x y z">
+    <link name="${parent}_counterweight_link">
+			<inertial>
+				<mass value="${m}"/>
+				<inertia ixx="0.000001" ixy="0" ixz="0" iyy="0.000001" iyz="0" izz="0.000001"/>
+			</inertial>
+		</link>
+    <joint name="${parent}_counterweight_joint" type="fixed">
+			<origin xyz="${x} ${y} ${z}" rpy="0 0 0"/>
+			<parent link="${parent}"/>
+			<child link="${parent}_counterweight_link"/>
+		</joint>
+	</xacro:macro>
 </robot>

File: stevie_description/urdf/stevie.xacro (robot description, xacro)
@@ -14,4 +14,5 @@
   <!-- DEPENDENCIES -->
   <xacro:include filename="$(find stevie_description)/urdf/macros.xacro" />
+  <xacro:include filename="$(find stevie_description)/urdf/materials.xacro" />
   <xacro:include filename="$(find stevie_description)/urdf/stevie.gazebo"/>
   <xacro:include filename="$(find stevie_description)/urdf/sensors/sensor_macros.xacro"/>

File: stevie_description/urdf/upper_body/hip.xacro (robot description, xacro)
@@ -3,5 +3,5 @@
 	<xacro:include filename="$(find stevie_description)/urdf/upper_body/upper_body.transmission.xacro" />
 	<!-- DECLARE VARIABLES -->
-	<xacro:property name="hip_mass" value="0.1"/>
+	<xacro:property name="hip_mass" value="0.5"/>
 	<xacro:property name="hip_volume" value="0.001004"/>
 	<xacro:property name="hip_length" value="0.320"/>
@@ -24,7 +24,7 @@
 			<visual>
 				<origin xyz="0 0 0" rpy="0 0 0"/>
-					<geometry>
-				 		<mesh filename="package://stevie_description/meshes/visual/hip_upper.stl" scale="0.001 0.001 0.001"/>
-					</geometry>
+				<geometry>
+			 		<mesh filename="package://stevie_description/meshes/visual/hip_upper.stl" scale="0.001 0.001 0.001"/>
+				</geometry>
 			</visual>
 			<inertial>

File: stevie_description/urdf/upper_body/upper_body.xacro (robot description, xacro)
@@ -4,5 +4,5 @@
 	<xacro:include filename="$(find stevie_description)/urdf/upper_body/hip.xacro" />
 	<!-- DECLARE VARIABLES -->
-	<xacro:property name="upper_body_mass" value="8"/>
+	<xacro:property name="upper_body_mass" value="0.8"/>
 	<xacro:property name="upper_body_volume" value="0.010712"/>
 	<xacro:property name="upper_body_length" value="0.347374786"/>
@@ -28,7 +28,9 @@
 			</visual>
 			<inertial>
-				<origin xyz="${upper_body_center_of_mass}" rpy="0 0 0"/>
+				<!--origin xyz="${upper_body_center_of_mass}" rpy="0 0 0"/-->
+				<origin xyz="0 0 ${upper_body_height/2}" rpy="0 0 0"/>
 				<mass value="${upper_body_mass}"/>
-				<xacro:scale_inertia m="${upper_body_mass}" v="${upper_body_volume}" ixx="0.0001825920" ixy="0" ixz="0" iyy="0.0001372321" iyz="0" izz="0.0001830431"/>
+				<!--xacro:scale_inertia m="${upper_body_mass}" v="${upper_body_volume}" ixx="0.0001825920" ixy="0" ixz="0" iyy="0.0001372321" iyz="0" izz="0.0001830431"/-->
+				<xacro:box_inertia m="${upper_body_mass}" x="${upper_body_width}" y="${upper_body_length}" z="${upper_body_height}"/>
 			</inertial>
 		</link>
@@ -48,5 +50,5 @@
 			<parent link="hip_link"/>
 			<child link="${name}_link"/>
-      <dynamics damping="10" friction="1.5"/>
+      <dynamics damping="100" friction="0.5"/>
 		</joint>
 		<!-- transmission -->

File: stevie_description/urdf/wheels/wheels.xacro (robot description, xacro)
@@ -35,8 +35,8 @@
 			<mu1>1.0</mu1>
 			<mu2>1.0</mu2>
-			<kp value="10000000.0"/>
-      <kd value="1.0"/>
-      <fdir1 value="1 0 0"/>
-			<maxVel>0</maxVel>
+			<!--kp value="10000000.0"/>
+      <kd value="100.0"/>
+			<minDepth>0.001</minDepth>
+			<maxVel>1.0</maxVel-->
 			<material>Gazebo/Black</material>
 		</gazebo>
@@ -54,5 +54,5 @@
 			<child link="wheel_${side}_link"/>
       <limit effort="100" velocity="100"/>
-      <dynamics damping="0.0" friction="0.5"/>
+      <dynamics damping="1.0" friction="0.5"/>
 		</joint>
 		<!-- transmission -->
