Commit message: Caster wheel added

File: stevie_description/urdf/lower_body/lower_body.xacro (robot description, xacro)
@@ -5,4 +5,5 @@
 -->
 	<xacro:include filename="$(find stevie_description)/urdf/wheels/wheels.xacro" />
+	<xacro:include filename="$(find stevie_description)/urdf/caster/caster.xacro" />
 	<!-- DECLARE VARIABLES -->
 	<xacro:property name="lower_body_mass" value="0.27"/>
@@ -10,5 +11,5 @@
 	<xacro:property name="lower_body_width" value="0.516555237"/>
 	<xacro:property name="lower_body_height" value="0.475"/>
-	<xacro:property name="z_adjustment" value="-0.075"/>
+	<xacro:property name="lower_body_z_adjustment" value="-0.075"/>
 	<xacro:property name="PI" value="3.14159"/>
 	<!--************************        LOWER BODY          ************************-->
@@ -41,5 +42,5 @@
 		<!-- footprint-lower_body joint -->
 		<joint name="${name}_footprint_joint" type="fixed">
-			<origin xyz="0 0 ${z_adjustment}" rpy="${PI/2} 0 ${PI/2}"/>
+			<origin xyz="0 0 ${lower_body_z_adjustment}" rpy="${PI/2} 0 ${PI/2}"/>
 			<parent link="${name}_footprint"/>
 			<child link="${name}_link"/>
@@ -48,4 +49,6 @@
 		<xacro:wheel parent="${name}_footprint" side="right"/>
 		<xacro:wheel parent="${name}_footprint" side="left"/>
+		<!--**************        CASTER          **************-->
+		<xacro:caster parent="${name}_footprint"/>
 	</xacro:macro>
 	<!--***********************************************************************-->

Commit message: Added acceleration limits so the robot no longer falls when it stops + restored the previous center of inertia for the lower part

File: stevie_description/urdf/lower_body/lower_body.xacro (robot description, xacro)
@@ -12,6 +12,6 @@
 	<xacro:property name="lower_body_width" value="0.516555"/>
 	<xacro:property name="lower_body_height" value="0.475"/>
-	<!--xacro:property name="lower_body_center_of_mass" value="-0.112043 0.000001 0.051805"/-->
-	<xacro:property name="lower_body_center_of_mass" value="-0.212043 0.000001 0"/>
+	<xacro:property name="lower_body_center_of_mass" value="-0.112043 0.000001 0.051805"/>
+	<!--xacro:property name="lower_body_center_of_mass" value="-0.212043 0.000001 0"/-->
 	<xacro:property name="PI" value="3.14159"/>
 	<!--************************        LOWER BODY          ************************-->

Commit message: Added dependencies to build a map from a single laser

File: stevie_description/urdf/lower_body/lower_body.xacro (robot description, xacro)
@@ -18,5 +18,5 @@
   <xacro:macro name="lower_body" params="name" >
 		<!-- base link -->
-		<link name="${name}_footprint"/>
+		<link name="base_link"/>
 		<!-- lower body link -->
 		<link name="${name}_link">
@@ -48,5 +48,5 @@
 		<joint name="${name}_footprint_joint" type="fixed">
 			<origin xyz="0 0 0" rpy="0 0 0"/>
-			<parent link="${name}_footprint"/>
+			<parent link="base_link"/>
 			<child link="${name}_link"/>
 		</joint>
